File: OBC_Boards/STM32_Breakout/STM32_Breakout.sch (KiCad schematic (older format))
At the start: 32 parts, among them U2 STM32F446RETx

Commit message: Add new microcontroller that will be used. Add footprint and symbol for common resistors and capacitors Add VREF circuitry, VDDIO and VDDUSB circuit:wq
Parts:
- removed R2, R3, R7: 10k, Resistor_SMD:R_0402_1005Metric_Pad0.72x0.64mm_HandSolder, symbol Device:R_Small
- added C1: 1u, CAPC1608X90, symbol CC0603MRX5R5BB475:CC0603MRX5R5BB475
- added C2, C? (x2): 100n, CAPC1608X90, symbol CC0603MRX5R5BB475:CC0603MRX5R5BB475
- added FB2, FB?: 100 ohm @ 100 MHz, Inductor_SMD:L_0805_2012Metric_Pad1.05x1.20mm_HandSolder, symbol Device:Ferrite_Bead_Small
- added R2, R7: 10k, RESC1607X60N, symbol STM32_Breakout-rescue:R0603-OBC_Libary
- added R3, R4: 10k +-1%, RESC1607X60N, symbol STM32_Breakout-rescue:R0603-OBC_Libary
- added R5: 32.5k +-1%, RESC1607X60N, symbol STM32_Breakout-rescue:R0603-OBC_Libary
- added U3: STM32L4A6ZGT6P, LQFP144-20x20mm, symbol STM32L4A6ZGT6P:STM32L4A6ZGT6P
- gave numbers to parts that had none: 1
Connections:
- net labels added: GNDA, VDDIO2, VDDUSB
- wire segments 72 -> 109
Other:
- moved on the sheet: D3

Commit message: dd minor circuitry
Parts:
- removed C10, C11, C12, C13, C4, C5, C6, C7, C8, C9: 100nF, Capacitor_SMD:C_0402_1005Metric_Pad0.74x0.62mm_HandSolder, symbol Device:C_Small
- removed C14: 10nF, Capacitor_SMD:C_0402_1005Metric_Pad0.74x0.62mm_HandSolder, symbol Device:C_Small
- removed C3: 10uF, Capacitor_SMD:C_0805_2012Metric_Pad1.18x1.45mm_HandSolder, symbol Device:C_Small
- removed R1: 2k2, Resistor_SMD:R_0603_1608Metric_Pad0.98x0.95mm_HandSolder, symbol Device:R_Small
- added C1: 4.7u, CAPC1608X90, symbol CC0603MRX5R5BB475:CC0603MRX5R5BB475
- added C10, C12, C14, C16, C17, C2, C3, C4, C5, C6, C7, C8, C9: 100n, CAPC1608X90, symbol CC0603MRX5R5BB475:CC0603MRX5R5BB475
- added C11: 1u, CAPC1608X90, symbol CC0603MRX5R5BB475:CC0603MRX5R5BB475
- added FB4: 100R @ 100 MHz, Inductor_SMD:L_0805_2012Metric_Pad1.05x1.20mm_HandSolder, symbol Device:Ferrite_Bead_Small
- added R?: 2k2, RESC1607X60N, symbol STM32_Breakout-rescue:R0603-OBC_Libary
- C13, C15: renamed from C?; value 100n -> 4.7u
- FB1: renamed from FB2; value 100 ohm @ 100 MHz -> 100R @ 100 MHz
- gave numbers to parts that had none: 1
Connections:
- wire segments 109 -> 104
Other:
- moved on the sheet: D2, FB1, FB2, FB3, R4

Commit message: Add IR4301 to schematic
Parts:
- added U?: IR4301, Package_DFN_QFN:Infineon_PQFN-22-15-4EP_6x5mm_P0.65mm, symbol Amplifier_Audio:IR4301
- gave numbers to parts that had none: 1
Changed lines of the file:
@@
 Text GLabel 6650 7250 1    50   Input ~ 0
 BOOT0
-Text GLabel 6950 7250 1    50   Input ~ 0
-BOOT1
 $Comp
 L power:GND #PWR023
@@
 	5950 2700 5950 15300
 $Comp
-L power:+3.3VA #PWR?
+L power:+3.3VA #PWR0102
 U 1 1 61A893DE
 P 4250 5200
-F 0 "#PWR?" H 4250 5050 50  0001 C CNN
+F 0 "#PWR0102" H 4250 5050 50  0001 C CNN
 F 1 "+3.3VA" V 4150 5300 50  0000 C CNN
 F 2 "" H 4250 5200 50  0001 C CNN
@@
 	4350 4200 4300 4200
 $Comp
-L power:+3.3V #PWR?
+L power:+3.3V #PWR0103
 U 1 1 61A893F2
 P 4350 4200
-F 0 "#PWR?" H 4350 4050 50  0001 C CNN
+F 0 "#PWR0103" H 4350 4050 50  0001 C CNN
 F 1 "+3.3V" V 4400 4400 50  0000 C CNN
 F 2 "" H 4350 4200 50  0001 C CNN
@@
 Connection ~ 5100 5900
 $Comp
-L power:GND #PWR?
+L power:GND #PWR0104
 U 1 1 61B9EE09
 P 2250 5200
-F 0 "#PWR?" H 2250 4950 50  0001 C CNN
+F 0 "#PWR0104" H 2250 4950 50  0001 C CNN
 F 1 "GND" H 2255 5027 50  0000 C CNN
 F 2 "" H 2250 5200 50  0001 C CNN
@@
 Connection ~ 2250 4300
 $Comp
-L power:GNDA #PWR?
+L power:GNDA #PWR0105
 U 1 1 61C2EA9F
 P 2000 5400
-F 0 "#PWR?" H 2000 5150 50  0001 C CNN
+F 0 "#PWR0105" H 2000 5150 50  0001 C CNN
 F 1 "GNDA" H 2005 5227 50  0000 C CNN
 F 2 "" H 2000 5400 50  0001 C CNN
@@
 $EndComp
 $Comp
-L power:+3.3V #PWR?
+L power:+3.3V #PWR0106
 U 1 1 6192FA53
 P 2400 3750
-F 0 "#PWR?" H 2400 3600 50  0001 C CNN
+F 0 "#PWR0106" H 2400 3600 50  0001 C CNN
 F 1 "+3.3V" V 2450 3950 50  0000 C CNN
 F 2 "" H 2400 3750 50  0001 C CNN
@@
 	1400 3750 1150 3750
 $Comp
-L power:+3.3V #PWR?
+L power:+3.3V #PWR0107
 U 1 1 6196AF93
 P 1850 4500
-F 0 "#PWR?" H 1850 4350 50  0001 C CNN
+F 0 "#PWR0107" H 1850 4350 50  0001 C CNN
 F 1 "+3.3V" V 1900 4700 50  0000 C CNN
 F 2 "" H 1850 4500 50  0001 C CNN
@@
 	2250 5400 2000 5400
 $Comp
-L power:+3.3V #PWR?
+L power:+3.3V #PWR0108
 U 1 1 61990292
 P 2250 5600
-F 0 "#PWR?" H 2250 5450 50  0001 C CNN
+F 0 "#PWR0108" H 2250 5450 50  0001 C CNN
 F 1 "+3.3V" V 2150 5650 50  0000 C CNN
 F 2 "" H 2250 5600 50  0001 C CNN
@@
 Connection ~ 3900 2950
 $Comp
-L power:GND #PWR?
+L power:GND #PWR0109
 U 1 1 619FDB6E
 P 3900 3250
-F 0 "#PWR?" H 3900 3000 50  0001 C CNN
+F 0 "#PWR0109" H 3900 3000 50  0001 C CNN
 F 1 "GND" H 3905 3077 50  0000 C CNN
 F 2 "" H 3900 3250 50  0001 C CNN
@@
 $EndComp
 $Comp
-L power:GND #PWR?
+L power:GND #PWR0110
 U 1 1 61A00DD3
 P 3600 3250
-F 0 "#PWR?" H 3600 3000 50  0001 C CNN
+F 0 "#PWR0110" H 3600 3000 50  0001 C CNN
 F 1 "GND" H 3605 3077 50  0000 C CNN
 F 2 "" H 3600 3250 50  0001 C CNN
@@
 $EndComp
 $Comp
-L power:GND #PWR?
+L power:GND #PWR0111
 U 1 1 61A0127C
 P 3300 3250
-F 0 "#PWR?" H 3300 3000 50  0001 C CNN
+F 0 "#PWR0111" H 3300 3000 50  0001 C CNN
 F 1 "GND" H 3305 3077 50  0000 C CNN
 F 2 "" H 3300 3250 50  0001 C CNN
@@
 $EndComp
 $Comp
-L power:GND #PWR?
+L power:GND #PWR0112
 U 1 1 61A015D8
 P 3000 3250
-F 0 "#PWR?" H 3000 3000 50  0001 C CNN
+F 0 "#PWR0112" H 3000 3000 50  0001 C CNN
 F 1 "GND" H 3005 3077 50  0000 C CNN
 F 2 "" H 3000 3250 50  0001 C CNN
@@
 $EndComp
 $Comp
-L power:GND #PWR?
+L power:GND #PWR0113
 U 1 1 61A0501F
 P 2700 3250
-F 0 "#PWR?" H 2700 3000 50  0001 C CNN
+F 0 "#PWR0113" H 2700 3000 50  0001 C CNN
 F 1 "GND" H 2705 3077 50  0000 C CNN
 F 2 "" H 2700 3250 50  0001 C CNN
@@
 $EndComp
 $Comp
-L power:GND #PWR?
+L power:GND #PWR0114
 U 1 1 61A052FE
 P 2400 3250
-F 0 "#PWR?" H 2400 3000 50  0001 C CNN
+F 0 "#PWR0114" H 2400 3000 50  0001 C CNN
 F 1 "GND" H 2405 3077 50  0000 C CNN
 F 2 "" H 2400 3250 50  0001 C CNN
@@
 $EndComp
 $Comp
-L power:GND #PWR?
+L power:GND #PWR0115
 U 1 1 61A0573B
 P 2100 3250
-F 0 "#PWR?" H 2100 3000 50  0001 C CNN
+F 0 "#PWR0115" H 2100 3000 50  0001 C CNN
 F 1 "GND" H 2105 3077 50  0000 C CNN
 F 2 "" H 2100 3250 50  0001 C CNN
@@
 $EndComp
 $Comp
-L power:GND #PWR?
+L power:GND #PWR0116
 U 1 1 61A05A9E
 P 1750 3250
-F 0 "#PWR?" H 1750 3000 50  0001 C CNN
+F 0 "#PWR0116" H 1750 3000 50  0001 C CNN
 F 1 "GND" H 1755 3077 50  0000 C CNN
 F 2 "" H 1750 3250 50  0001 C CNN
@@
 $EndComp
 $Comp
-L power:GND #PWR?
+L power:GND #PWR0117
 U 1 1 61A05F45
 P 1400 3250
-F 0 "#PWR?" H 1400 3000 50  0001 C CNN
+F 0 "#PWR0117" H 1400 3000 50  0001 C CNN
 F 1 "GND" H 1405 3077 50  0000 C CNN
 F 2 "" H 1400 3250 50  0001 C CNN
@@
 $EndComp
 $Comp
-L power:GND #PWR?
+L power:GND #PWR0118
 U 1 1 61A06340
 P 1050 3250
-F 0 "#PWR?" H 1050 3000 50  0001 C CNN
+F 0 "#PWR0118" H 1050 3000 50  0001 C CNN
 F 1 "GND" H 1055 3077 50  0000 C CNN
 F 2 "" H 1050 3250 50  0001 C CNN
@@
 $EndComp
 $Comp
-L power:GND #PWR?
+L power:GND #PWR0119
 U 1 1 61A06734
 P 4250 3350
-F 0 "#PWR?" H 4250 3100 50  0001 C CNN
+F 0 "#PWR0119" H 4250 3100 50  0001 C CNN
 F 1 "GND" H 4255 3177 50  0000 C CNN
 F 2 "" H 4250 3350 50  0001 C CNN
@@
 $EndComp
 $Comp
-L STM32_Breakout-rescue:R0603-OBC_Libary R?
+L STM32_Breakout-rescue:R0603-OBC_Libary R1
 U 1 1 61A100BF
 P 4250 3150
-F 0 "R?" V 4200 3250 50  0000 L CNN
+F 0 "R1" V 4200 3250 50  0000 L CNN
 F 1 "2k2" V 4350 3200 50  0000 L CNN
 F 2 "RESC1607X60N" H 4200 3250 50  0001 L BNN
@@
 	1400 3750 1800 3750
 $Comp
-L power:GND #PWR?
+L power:GND #PWR0120
 U 1 1 61A4F0A0
 P 1400 4050
-F 0 "#PWR?" H 1400 3800 50  0001 C CNN
+F 0 "#PWR0120" H 1400 3800 50  0001 C CNN
 F 1 "GND" H 1405 3877 50  0000 C CNN
 F 2 "" H 1400 4050 50  0001 C CNN
@@
 $EndComp
 $Comp
-L power:GND #PWR?
+L power:GND #PWR0121
 U 1 1 61A53F74
 P 1800 4050
-F 0 "#PWR?" H 1800 3800 50  0001 C CNN
+F 0 "#PWR0121" H 1800 3800 50  0001 C CNN
 F 1 "GND" H 1805 3877 50  0000 C CNN
 F 2 "" H 1800 4050 50  0001 C CNN
@@
 	1550 4500 1650 4500
 $Comp
-L power:GND #PWR?
+L power:GND #PWR0122
 U 1 1 61A5E813
 P 1250 4800
-F 0 "#PWR?" H 1250 4550 50  0001 C CNN
+F 0 "#PWR0122" H 1250 4550 50  0001 C CNN
 F 1 "GND" H 1255 4627 50  0000 C CNN
 F 2 "" H 1250 4800 50  0001 C CNN
@@
 $EndComp
 $Comp
-L power:GND #PWR?
+L power:GND #PWR0123
 U 1 1 61A5ED60
 P 1550 4800
-F 0 "#PWR?" H 1550 4550 50  0001 C CNN
+F 0 "#PWR0123" H 1550 4550 50  0001 C CNN
 F 1 "GND" H 1555 4627 50  0000 C CNN
 F 2 "" H 1550 4800 50  0001 C CNN
@@
 $EndComp
 $Comp
-L power:GNDA #PWR?
+L power:GNDA #PWR0124
 U 1 1 61A62802
 P 4250 6000
-F 0 "#PWR?" H 4250 5750 50  0001 C CNN
+F 0 "#PWR0124" H 4250 5750 50  0001 C CNN
 F 1 "GNDA" H 4255 5827 50  0000 C CNN
 F 2 "" H 4250 6000 50  0001 C CNN
@@
 $EndComp
 $Comp
-L power:GNDA #PWR?
+L power:GNDA #PWR0125
 U 1 1 61A6336A
 P 4700 6200
-F 0 "#PWR?" H 4700 5950 50  0001 C CNN
+F 0 "#PWR0125" H 4700 5950 50  0001 C CNN
 F 1 "GNDA" H 4705 6027 50  0000 C CNN
 F 2 "" H 4700 6200 50  0001 C CNN
@@
 $EndComp
 $Comp
-L power:GNDA #PWR?
+L power:GNDA #PWR0126
 U 1 1 61A637E3
 P 5100 6200
-F 0 "#PWR?" H 5100 5950 50  0001 C CNN
+F 0 "#PWR0126" H 5100 5950 50  0001 C CNN
 F 1 "GNDA" H 5105 6027 50  0000 C CNN
 F 2 "" H 5100 6200 50  0001 C CNN
@@
 $EndComp
 $Comp
-L power:GNDA #PWR?
+L power:GNDA #PWR0127
 U 1 1 61A63D2A
 P 5350 6350
-F 0 "#PWR?" H 5350 6100 50  0001 C CNN
+F 0 "#PWR0127" H 5350 6100 50  0001 C CNN
 F 1 "GNDA" H 5355 6177 50  0000 C CNN
 F 2 "" H 5350 6350 50  0001 C CNN
@@
 Connection ~ 2200 3750
 $Comp
-L power:GND #PWR?
+L power:GND #PWR0128
 U 1 1 61A708A2
 P 2200 4050
-F 0 "#PWR?" H 2200 3800 50  0001 C CNN
+F 0 "#PWR0128" H 2200 3800 50  0001 C CNN
 F 1 "GND" H 2050 3950 50  0000 C CNN
 F 2 "" H 2200 4050 50  0001 C CNN
@@
 $EndComp
 $Comp
-L power:+3.3V #PWR?
+L power:+3.3V #PWR0129
 U 1 1 61B88B56
 P 5200 5300
-F 0 "#PWR?" H 5200 5150 50  0001 C CNN
+F 0 "#PWR0129" H 5200 5150 50  0001 C CNN
 F 1 "+3.3V" H 5250 5500 50  0000 C CNN
 F 2 "" H 5200 5300 50  0001 C CNN
@@
 Wire Wire Line
 	5200 5900 5350 5900
+Text GLabel 6950 7250 1    50   Input ~ 0
+BOOT1
+$Comp
+L Amplifier_Audio:IR4301 U?
+U 1 1 61984E96
+P 8300 5350
+F 0 "U?" H 8300 6331 50  0000 C CNN
+F 1 "IR4301" H 8300 6240 50  0000 C CNN
+F 2 "Package_DFN_QFN:Infineon_PQFN-22-15-4EP_6x5mm_P0.65mm" H 8300 5350 50  0001 C CIN
+F 3 "https://www.infineon.com/dgdl/ir4301.pdf?fileId=5546d462533600a4015355d5fc691819" H 8300 5350 50  0001 C CNN
+	1    8300 5350
+	1    0    0    -1
+$EndComp
 $EndSCHEMATC

Commit message: Added power monitor circuit
Still not sure if amp's footnote is updated
Parts:
- added CurSense1: 20m, symbol Device:R
- added IC1: MAX4372F, Max4372FESA+:MAX4372FESA&plus_, symbol MAX4372HEUK+T:MAX4372HEUK+T
- C1, C10, C11, C12, C13, C14, C15, C16, C17, C2, C3, C4, C5, C6, C7, C8, C9: symbol CC0603MRX5R5BB475:CC0603MRX5R5BB475 -> STM32_Breakout-rescue:CC0603MRX5R5BB475-CC0603MRX5R5BB475
- U1: symbol STM32L4R5ZIT6P:STM32L4R5ZIT6P -> STM32_Breakout-rescue:STM32L4R5ZIT6P-STM32L4R5ZIT6P
- U3: symbol STM32L4A6ZGT6P:STM32L4A6ZGT6P -> STM32_Breakout-rescue:STM32L4A6ZGT6P-STM32L4A6ZGT6P
- gave numbers to parts that had none: 1
Connections:
- net labels added: PIN, STM32_VCC
- wire segments 104 -> 110
Changed lines of the file:
@@
 Temperature Sensor
 $Comp
-L STM32L4R5ZIT6P:STM32L4R5ZIT6P U1
+L STM32_Breakout-rescue:STM32L4R5ZIT6P-STM32L4R5ZIT6P U1
 U 1 1 617E0C56
 P -10800 5500
@@
 Memory
 $Comp
-L STM32L4A6ZGT6P:STM32L4A6ZGT6P U3
+L STM32_Breakout-rescue:STM32L4A6ZGT6P-STM32L4A6ZGT6P U3
 U 1 1 61927926
 P 2000 7100
@@
 $EndComp
 $Comp
-L STM32L4A6ZGT6P:STM32L4A6ZGT6P U3
+L STM32_Breakout-rescue:STM32L4A6ZGT6P-STM32L4A6ZGT6P U3
 U 3 1 6193793B
 P 2250 4200
@@
 $EndComp
 $Comp
-L STM32L4A6ZGT6P:STM32L4A6ZGT6P U3
+L STM32_Breakout-rescue:STM32L4A6ZGT6P-STM32L4A6ZGT6P U3
 U 2 1 6191DFF4
 P 1900 11400
@@
 	4300 4700 4300 4800
 $Comp
-L CC0603MRX5R5BB475:CC0603MRX5R5BB475 C1
+L STM32_Breakout-rescue:CC0603MRX5R5BB475-CC0603MRX5R5BB475 C1
 U 1 1 61AD676F
 P 4700 6000
@@
 $EndComp
 $Comp
-L CC0603MRX5R5BB475:CC0603MRX5R5BB475 C2
+L STM32_Breakout-rescue:CC0603MRX5R5BB475-CC0603MRX5R5BB475 C2
 U 1 1 61AF06E3
 P 5100 6000
@@
 $EndComp
 $Comp
-L CC0603MRX5R5BB475:CC0603MRX5R5BB475 C13
+L STM32_Breakout-rescue:CC0603MRX5R5BB475-CC0603MRX5R5BB475 C13
 U 1 1 61953FC5
 P 1400 3850
@@
 $EndComp
 $Comp
-L CC0603MRX5R5BB475:CC0603MRX5R5BB475 C15
+L STM32_Breakout-rescue:CC0603MRX5R5BB475-CC0603MRX5R5BB475 C15
 U 1 1 6196AFA0
 P 1250 4600
@@
 	1100 4500 1250 4500
 $Comp
-L CC0603MRX5R5BB475:CC0603MRX5R5BB475 C16
+L STM32_Breakout-rescue:CC0603MRX5R5BB475-CC0603MRX5R5BB475 C16
 U 1 1 619B160E
 P 1550 4600
@@
 $EndComp
 $Comp
-L CC0603MRX5R5BB475:CC0603MRX5R5BB475 C2
+L STM32_Breakout-rescue:CC0603MRX5R5BB475-CC0603MRX5R5BB475 C2
 U 1 1 619B36B1
 P 1400 3050
@@
 $EndComp
 $Comp
-L CC0603MRX5R5BB475:CC0603MRX5R5BB475 C1
+L STM32_Breakout-rescue:CC0603MRX5R5BB475-CC0603MRX5R5BB475 C1
 U 1 1 619CBE03
 P 1050 3050
@@
 	1050 2950 1400 2950
 $Comp
-L CC0603MRX5R5BB475:CC0603MRX5R5BB475 C3
+L STM32_Breakout-rescue:CC0603MRX5R5BB475-CC0603MRX5R5BB475 C3
 U 1 1 619D8077
 P 1750 3050
@@
 $EndComp
 $Comp
-L CC0603MRX5R5BB475:CC0603MRX5R5BB475 C4
+L STM32_Breakout-rescue:CC0603MRX5R5BB475-CC0603MRX5R5BB475 C4
 U 1 1 619DEB7C
 P 2100 3050
@@
 	2100 2950 2400 2950
 $Comp
-L CC0603MRX5R5BB475:CC0603MRX5R5BB475 C5
+L STM32_Breakout-rescue:CC0603MRX5R5BB475-CC0603MRX5R5BB475 C5
 U 1 1 619E8B20
 P 2400 3050
@@
 	2400 2950 2700 2950
 $Comp
-L CC0603MRX5R5BB475:CC0603MRX5R5BB475 C6
+L STM32_Breakout-rescue:CC0603MRX5R5BB475-CC0603MRX5R5BB475 C6
 U 1 1 619E9002
 P 2700 3050
@@
 	2700 2950 3000 2950
 $Comp
-L CC0603MRX5R5BB475:CC0603MRX5R5BB475 C7
+L STM32_Breakout-rescue:CC0603MRX5R5BB475-CC0603MRX5R5BB475 C7
 U 1 1 619E9366
 P 3000 3050
@@
 	3000 2950 3300 2950
 $Comp
-L CC0603MRX5R5BB475:CC0603MRX5R5BB475 C8
+L STM32_Breakout-rescue:CC0603MRX5R5BB475-CC0603MRX5R5BB475 C8
 U 1 1 619E97C6
 P 3300 3050
@@
 	3300 2950 3600 2950
 $Comp
-L CC0603MRX5R5BB475:CC0603MRX5R5BB475 C9
+L STM32_Breakout-rescue:CC0603MRX5R5BB475-CC0603MRX5R5BB475 C9
 U 1 1 619E9C28
 P 3600 3050
@@
 $EndComp
 $Comp
-L CC0603MRX5R5BB475:CC0603MRX5R5BB475 C10
+L STM32_Breakout-rescue:CC0603MRX5R5BB475-CC0603MRX5R5BB475 C10
 U 1 1 619F3EBD
 P 3900 3050
@@
 $EndComp
 $Comp
-L CC0603MRX5R5BB475:CC0603MRX5R5BB475 C11
+L STM32_Breakout-rescue:CC0603MRX5R5BB475-CC0603MRX5R5BB475 C11
 U 1 1 61A2BCAE
 P 5200 3400
@@
 $EndComp
 $Comp
-L CC0603MRX5R5BB475:CC0603MRX5R5BB475 C12
+L STM32_Breakout-rescue:CC0603MRX5R5BB475-CC0603MRX5R5BB475 C12
 U 1 1 61A31429
 P 5600 3400
@@
 $EndComp
 $Comp
-L CC0603MRX5R5BB475:CC0603MRX5R5BB475 C14
+L STM32_Breakout-rescue:CC0603MRX5R5BB475-CC0603MRX5R5BB475 C14
 U 1 1 61A43B77
 P 1800 3850
@@
 $EndComp
 $Comp
-L CC0603MRX5R5BB475:CC0603MRX5R5BB475 C17
+L STM32_Breakout-rescue:CC0603MRX5R5BB475-CC0603MRX5R5BB475 C17
 U 1 1 61A69F57
 P 2200 3850
@@
 BOOT1
 $Comp
-L Amplifier_Audio:IR4301 U?
+L Amplifier_Audio:IR4301 U4
 U 1 1 61984E96
 P 8300 5350
-F 0 "U?" H 8300 6331 50  0000 C CNN
+F 0 "U4" H 8300 6331 50  0000 C CNN
 F 1 "IR4301" H 8300 6240 50  0000 C CNN
 F 2 "Package_DFN_QFN:Infineon_PQFN-22-15-4EP_6x5mm_P0.65mm" H 8300 5350 50  0001 C CIN
@@
 	1    0    0    -1
 $EndComp
+$Comp
+L MAX4372HEUK+T:MAX4372HEUK+T IC1
+U 1 1 619C7D9D
+P 1050 1900
+F 0 "IC1" H 1550 2165 50  0000 C CNN
+F 1 "MAX4372F" H 1550 2074 50  0000 C CNN
+F 2 "Max4372FESA+:MAX4372FESA&plus_" H 1900 2000 50  0001 L CNN
+F 3 "https://componentsearchengine.com/Datasheets/2/MAX4372HEUK+T.pdf" H 1900 1900 50  0001 L CNN
+F 4 "Maxim MAX4372HEUK+T, Current Sensing Amplifier Single 5-Pin SOT-23" H 1900 1800 50  0001 L CNN "Description"
+F 5 "1.45" H 1900 1700 50  0001 L CNN "Height"
+F 6 "Maxim Integrated" H 1900 1600 50  0001 L CNN "Manufacturer_Name"
+F 7 "MAX4372HEUK+T" H 1900 1500 50  0001 L CNN "Manufacturer_Part_Number"
+F 8 "700-MAX4372HEUK+T" H 1900 1400 50  0001 L CNN "Mouser Part Number"
+F 9 "https://www.mouser.co.uk/ProductDetail/Maxim-Integrated/MAX4372HEUK%2bT?qs=1eQvB6Dk1vguheoXjIjTiA%3D%3D" H 1900 1300 50  0001 L CNN "Mouser Price/Stock"
+F 10 "" H 1900 1200 50  0001 L CNN "Arrow Part Number"
+F 11 "" H 1900 1100 50  0001 L CNN "Arrow Price/Stock"
+	1    1050 1900
+	1    0    0    -1
+$EndComp
+$Comp
+L power:GND #PWR0130
+U 1 1 619D71B4
+P 1050 1900
+F 0 "#PWR0130" H 1050 1650 50  0001 C CNN
+F 1 "GND" H 1055 1727 50  0000 C CNN
+F 2 "" H 1050 1900 50  0001 C CNN
+F 3 "" H 1050 1900 50  0001 C CNN
+	1    1050 1900
+	0    1    1    0
+$EndComp
+$Comp
+L power:VCC #PWR0131
+U 1 1 619DAC3A
+P 1050 2100
+F 0 "#PWR0131" H 1050 1950 50  0001 C CNN
+F 1 "VCC" H 1065 2273 50  0000 C CNN
+F 2 "" H 1050 2100 50  0001 C CNN
+F 3 "" H 1050 2100 50  0001 C CNN
+	1    1050 2100
+	0    -1   -1   0
+$EndComp
+Text GLabel 1050 2000 0    50   Input ~ 0
+PIN
+$Comp
+L Device:R CurSense1
+U 1 1 619E1C1F
+P 2350 1950
+F 0 "CurSense1" H 2420 1996 50  0000 L CNN
+F 1 "20m" H 2420 1905 50  0000 L CNN
+F 2 "" V 2280 1950 50  0001 C CNN
+F 3 "~" H 2350 1950 50  0001 C CNN
+	1    2350 1950
+	1    0    0    -1
+$EndComp
+Wire Wire Line
+	2050 1900 2050 1800
+Wire Wire Line
+	2050 1800 2350 1800
+Wire Wire Line
+	2050 2000 2050 2100
+Wire Wire Line
+	2050 2100 2350 2100
+Wire Wire Line
+	2350 1800 2350 1700
+Connection ~ 2350 1800
+Wire Wire Line
+	2350 2100 2350 2200
+Connection ~ 2350 2100
+Text GLabel 2350 2200 2    50   Input ~ 0
+STM32_VCC
+$Comp
+L power:VCC #PWR0132
+U 1 1 61A0B1CB
+P 2350 1700
+F 0 "#PWR0132" H 2350 1550 50  0001 C CNN
+F 1 "VCC" H 2365 1873 50  0000 C CNN
+F 2 "" H 2350 1700 50  0001 C CNN
+F 3 "" H 2350 1700 50  0001 C CNN
+	1    2350 1700
+	1    0    0    -1
+$EndComp

Commit message: Added power monitor to circuit
Added 8-pin max4372F (amplifies by 50 times) with corresponding footnote and current sensing resistor. Out voltage should have 0.3-3.0 V range
Parts:
- removed IC1: MAX4372F, Max4372FESA+:MAX4372FESA&plus_, symbol MAX4372HEUK+T:MAX4372HEUK+T
- added MAX4372F: MAX4372FESA+, Max4372FESA+:SOIC127P600X175-8N, symbol MAX4372FESA+:MAX4372FESA+
- CurSense1: value 20m -> 20mO
Connections:
- wire segments 110 -> 111
Changed lines of the file:
@@
 	1    0    0    -1
 $EndComp
-$Comp
-L MAX4372HEUK+T:MAX4372HEUK+T IC1
-U 1 1 619C7D9D
-P 1050 1900
-F 0 "IC1" H 1550 2165 50  0000 C CNN
-F 1 "MAX4372F" H 1550 2074 50  0000 C CNN
-F 2 "Max4372FESA+:MAX4372FESA&plus_" H 1900 2000 50  0001 L CNN
-F 3 "https://componentsearchengine.com/Datasheets/2/MAX4372HEUK+T.pdf" H 1900 1900 50  0001 L CNN
-F 4 "Maxim MAX4372HEUK+T, Current Sensing Amplifier Single 5-Pin SOT-23" H 1900 1800 50  0001 L CNN "Description"
-F 5 "1.45" H 1900 1700 50  0001 L CNN "Height"
-F 6 "Maxim Integrated" H 1900 1600 50  0001 L CNN "Manufacturer_Name"
-F 7 "MAX4372HEUK+T" H 1900 1500 50  0001 L CNN "Manufacturer_Part_Number"
-F 8 "700-MAX4372HEUK+T" H 1900 1400 50  0001 L CNN "Mouser Part Number"
-F 9 "https://www.mouser.co.uk/ProductDetail/Maxim-Integrated/MAX4372HEUK%2bT?qs=1eQvB6Dk1vguheoXjIjTiA%3D%3D" H 1900 1300 50  0001 L CNN "Mouser Price/Stock"
-F 10 "" H 1900 1200 50  0001 L CNN "Arrow Part Number"
-F 11 "" H 1900 1100 50  0001 L CNN "Arrow Price/Stock"
-	1    1050 1900
-	1    0    0    -1
-$EndComp
-$Comp
-L power:GND #PWR0130
-U 1 1 619D71B4
-P 1050 1900
-F 0 "#PWR0130" H 1050 1650 50  0001 C CNN
-F 1 "GND" H 1055 1727 50  0000 C CNN
-F 2 "" H 1050 1900 50  0001 C CNN
-F 3 "" H 1050 1900 50  0001 C CNN
-	1    1050 1900
-	0    1    1    0
-$EndComp
-$Comp
-L power:VCC #PWR0131
-U 1 1 619DAC3A
-P 1050 2100
-F 0 "#PWR0131" H 1050 1950 50  0001 C CNN
-F 1 "VCC" H 1065 2273 50  0000 C CNN
-F 2 "" H 1050 2100 50  0001 C CNN
-F 3 "" H 1050 2100 50  0001 C CNN
-	1    1050 2100
-	0    -1   -1   0
-$EndComp
-Text GLabel 1050 2000 0    50   Input ~ 0
-PIN
-$Comp
-L Device:R CurSense1
-U 1 1 619E1C1F
-P 2350 1950
-F 0 "CurSense1" H 2420 1996 50  0000 L CNN
-F 1 "20m" H 2420 1905 50  0000 L CNN
-F 2 "" V 2280 1950 50  0001 C CNN
-F 3 "~" H 2350 1950 50  0001 C CNN
-	1    2350 1950
-	1    0    0    -1
-$EndComp
-Wire Wire Line
-	2050 1900 2050 1800
-Wire Wire Line
-	2050 1800 2350 1800
-Wire Wire Line
-	2050 2000 2050 2100
-Wire Wire Line
-	2050 2100 2350 2100
-Wire Wire Line
-	2350 1800 2350 1700
-Connection ~ 2350 1800
-Wire Wire Line
-	2350 2100 2350 2200
-Connection ~ 2350 2100
-Text GLabel 2350 2200 2    50   Input ~ 0
+Text GLabel 3450 2150 2    50   Input ~ 0
 STM32_VCC
 $Comp
 L power:VCC #PWR0132
 U 1 1 61A0B1CB
-P 2350 1700
-F 0 "#PWR0132" H 2350 1550 50  0001 C CNN
-F 1 "VCC" H 2365 1873 50  0000 C CNN
-F 2 "" H 2350 1700 50  0001 C CNN
-F 3 "" H 2350 1700 50  0001 C CNN
-	1    2350 1700
+P 3450 1650
+F 0 "#PWR0132" H 3450 1500 50  0001 C CNN
+F 1 "VCC" H 3465 1823 50  0000 C CNN
+F 2 "" H 3450 1650 50  0001 C CNN
+F 3 "" H 3450 1650 50  0001 C CNN
+	1    3450 1650
 	1    0    0    -1
 $EndComp
+Wire Wire Line
+	3450 2050 3450 2150
+Connection ~ 3450 1750
+Wire Wire Line
+	3450 1750 3450 1650
+Wire Wire Line
+	3150 1750 3250 1750
+$Comp
+L Device:R CurSense1
+U 1 1 619E1C1F
+P 3450 1900
+F 0 "CurSense1" H 3520 1946 50  0000 L CNN
+F 1 "20mO" H 3520 1855 50  0000 L CNN
+F 2 "" V 3380 1900 50  0001 C CNN
+F 3 "~" H 3450 1900 50  0001 C CNN
+	1    3450 1900
+	1    0    0    -1
+$EndComp
+Text GLabel 1050 2050 0    50   Input ~ 0
+PIN
+$Comp
+L power:VCC #PWR0131
+U 1 1 619DAC3A
+P 1050 1750
+F 0 "#PWR0131" H 1050 1600 50  0001 C CNN
+F 1 "VCC" H 1065 1923 50  0000 C CNN
+F 2 "" H 1050 1750 50  0001 C CNN
+F 3 "" H 1050 1750 50  0001 C CNN
+	1    1050 1750
+	0    -1   -1   0
+$EndComp
+$Comp
+L MAX4372FESA+:MAX4372FESA+ MAX4372F
+U 1 1 61A27419
+P 1050 1750
+F 0 "MAX4372F" H 2150 2137 60  0000 C CNN
+F 1 "MAX4372FESA+" H 2150 2031 60  0000 C CNN
+F 2 "Max4372FESA+:SOIC127P600X175-8N" H 2150 1990 60  0001 C CNN
+F 3 "" H 1050 1750 60  0000 C CNN
+	1    1050 1750
+	1    0    0    -1
+$EndComp
+Connection ~ 3250 1750
+Wire Wire Line
+	3250 1750 3450 1750
+$Comp
+L power:GND #PWR0130
+U 1 1 619D71B4
+P 1050 1950
+F 0 "#PWR0130" H 1050 1700 50  0001 C CNN
+F 1 "GND" H 1055 1777 50  0000 C CNN
+F 2 "" H 1050 1950 50  0001 C CNN
+F 3 "" H 1050 1950 50  0001 C CNN
+	1    1050 1950
+	0    1    1    0
+$EndComp
+Wire Wire Line
+	3250 1950 3350 1950
+Wire Wire Line
+	3350 1950 3350 2050
+Wire Wire Line
+	3350 2050 3450 2050
+Connection ~ 3450 2050
 $EndSCHEMATC
