File: OBC_Boards/STM32_Breakout/STM32_Breakout.kicad_sch (KiCad schematic)
At the start: 96 parts, among them J1 Conn_02x20_Odd_Even, J2 ST1W008S4ER1500-MicroSDConnec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, J3 1050171001, J4 105017-1001, J5 1050171001, J6 SSQ-105-03-T-D, J7 SSQ-105-03-T-D, Q1 Q_PMOS_DGS, U1 MR25H10MDF, U2 BU33SA5WGWZ-E2-qsat-symb, U3 STM32L4A6ZGT6P, U4 MCP7940NT-I_MS, U5 FSM6JSMATR, U6 MCP9808

Commit message: Moved USB connector up
Parts:
- added S1: GF-123-0054, SW_GF-123-0054, symbol GF-123:GF-123-0054
- renumbered C28 to C1, C1 to C10, C17 to C11, C2 to C12, C3 to C13, C4 to C14, C5 to C15, C6 to C16, C7 to C17, C8 to C18, C9 to C19, C11 to C2, C22 to C20, C18 to C21, C10 to C22, C19 to C23, C23 to C26, C20 to C27, C21 to C28, C27 to C3, C26 to C4, C12 to C5, C15 to C6, C13 to C7, C16 to C8, C14 to C9, D7 to D1, D6 to D2, D1 to D3, D3 to D4, D2 to D5, D4 to D6, D5 to D7, FB10 to FB1, FB6 to FB10, FB1 to FB2, FB5 to FB3, FB9 to FB4, FB7 to FB5, FB2 to FB6, FB3 to FB7, FB4 to FB8, FB8 to FB9, J3 to J2, J5 to J3, J6 to J5, J7 to J6, J2 to J7, R10 to R1, R4 to R10, R5 to R11, R19 to R12, R20 to R13, R11 to R14, R12 to R15, R17 to R16, R13 to R17, R14 to R18, R15 to R19, R24 to R2, R21 to R20, R16 to R21, R9 to R23, R3 to R24, R8 to R25, R2 to R26, R23 to R3, R7 to R4, R18 to R5, R25 to R6, R26 to R7, R6 to R8, R1 to R9, U4 to U1, U6 to U2, U2 to U3, U3 to U4, U1 to U6
Connections:
- net BOOT1: now also S1.1; no longer R24.1
- net SPI2_NSS: no longer J1.26 (Pin_26)
- net SPI2_NSS2: now reaches U4.114 (PD0)
- net SPI2_NSS2: now also J1.26 (Pin_26)
- new net: R24.1, S1.2

Commit message: Add all old footprints to new schematic Add usb input with usb-uart interfacing to provide manual commands using uart
Parts:
- removed BT1: Battery_Cell, STM32_Breakout:36-3000-ND, symbol Device:Battery_Cell
- removed R23: 10k +-1%, RESC1607X60N, symbol STM32_Breakout-rescue:R0603-OBC_Libary
- added C29: 4.7u, CAPC1608X90, symbol STM32_Breakout-rescue:CC0603MRX5R5BB475-CC0603MRX5R5BB475
- added C30, C31, C32: 100n, CAPC1608X90, symbol STM32_Breakout-rescue:CC0603MRX5R5BB475-CC0603MRX5R5BB475
- added C33, C34: 47pF, CAPC1608X90, symbol STM32_Breakout-rescue:CC0603MRX5R5BB475-CC0603MRX5R5BB475
- added D10, D9: GREEN, LED_SMD:LED_0603_1608Metric_Pad1.05x0.95mm_HandSolder, symbol Device:LED_Small
- added D8: RED, LED_SMD:LED_0603_1608Metric_Pad1.05x0.95mm_HandSolder, symbol Device:LED_Small
- added FB11: 100R @ 100 MHz, STM32_Breakout:INDUC1607X60N, symbol Device:Ferrite_Bead_Small
- added J8: 105017-1001, STM32_Breakout:MOLEX_105017-1001, symbol STM32_Breakout-rescue:105017-1001-Imported_OBC_Library
- added R27, R30, R31: 2k2, RESC1607X60N, symbol STM32_Breakout-rescue:R0603-OBC_Libary
- added R28, R29: 27, RESC1607X60N, symbol STM32_Breakout-rescue:R0603-OBC_Libary
- added R32: 0R, RESC1607X60N, symbol STM32_Breakout-rescue:R0603-OBC_Libary
- added U7: FT231XS-R, SOP63P599X175-20N, symbol OBC_Library:FT231XS-R
Connections:
- net BOOT1 is gone; now on net +3V3: S1.1
- net +3V3: now also U1.3 (Vbat), FB11.1, R30.2, R31.2
- net BOOT0: now also R24.1, S1.2, U4.138 (PH3-BOOT0)
- net GND: now also J4.4, C29.1, C30.1, C31.1, C32.1, C33.1, C34.2, J8.4, J8.5, R27.2, R32.2, U7.16 (GND), U7.6 (GND)
- net LPUART1_CTS: now reaches U4.90 (PG5)
- net LPUART1_CTS: now also U7.2 (~{RTS})
- net LPUART1_RTS: now reaches U4.91 (PG6)
- net LPUART1_RTS: now also U7.9 (~{CTS})
- net LPUART1_TX: now reaches U4.92 (PG7)
- net LPUART1_TX: now also U7.4 (RXD)
- net LPUART1_RX: now reaches U4.93 (PG8)
- net LPUART1_RX: now also U7.20 (TXD)
- new net: C29.2, C30.2, C31.2, D8.2 (A), FB11.2, U7.15 (VCC)
- new net: C34.1, J8.2, R29.2
- new net: R28.1, U7.11 (USBDP)
- new net: C33.2, J8.3, R28.2
- new net: D10.1 (K), U7.10 (CBUS2)
- new net: D10.2 (A), R31.1
- new net: D9.2 (A), R30.1
- new net: C32.2, U7.13 (3V3OUT), U7.14 (~{RESET}), U7.3 (VCCIO)
- new net: D8.1 (K), R27.1
- new net: J8.S1 (SHIELD), J8.S2 (SHIELD), J8.S3 (SHIELD), J8.S4 (SHIELD), J8.S5 (SHIELD), J8.S6 (SHIELD), R32.1
- new net: R29.1, U7.12 (USBDM)
- new net: D9.1 (K), U7.17 (CBUS1)
- no-connect marks 5 -> 21
Other:
- note added: "Micro-USB Communication Port"
- moved on the sheet: S1

Commit message: Minor changes to schematic to make it more readable
Connections:
- net at J8.2, R29.2: no longer C34.1
- net at C33.2, J8.3, R28.2: now also C34.1
Other:
- moved on the sheet: C34
Changed lines of the file:
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@@
   (junction (at 80.01 101.6) (diameter 0) (color 0 0 0 0)
   )
-  (junction (at 478.79 165.1) (diameter 0) (color 0 0 0 0)
-  )
   (junction (at 55.88 101.6) (diameter 0) (color 0 0 0 0)
   )
@@
   (junction (at 271.78 80.01) (diameter 0) (color 0 0 0 0)
   )
+  (junction (at 471.17 162.56) (diameter 0) (color 0 0 0 0)
+  )
   (junction (at 68.58 38.1) (diameter 0) (color 0 0 0 0)
   )
@@
     (stroke (width 0) (type default) (color 0 0 0 0))
   )
-  (wire (pts (xy 457.2 162.56) (xy 481.33 162.56))
+  (wire (pts (xy 457.2 162.56) (xy 471.17 162.56))
     (stroke (width 0) (type default) (color 0 0 0 0))
   )
@@
     (stroke (width 0) (type default) (color 0 0 0 0))
   )
+  (wire (pts (xy 471.17 162.56) (xy 481.33 162.56))
+    (stroke (width 0) (type default) (color 0 0 0 0))
+  )
   (polyline (pts (xy 19.05 137.16) (xy 109.22 137.16))
     (stroke (width 0) (type default) (color 0 0 0 0))
@@
     (pin "2")
   )
-  (symbol (lib_id "STM32_Breakout-rescue:CC0603MRX5R5BB475-CC0603MRX5R5BB475") (at 478.79 170.18 270) (mirror x) (unit 1)
+  (symbol (lib_id "STM32_Breakout-rescue:CC0603MRX5R5BB475-CC0603MRX5R5BB475") (at 471.17 157.48 90) (mirror x) (unit 1)
     (in_bom yes) (on_board yes)
-    (property "Reference" "C34" (id 0) (at 482.6 171.45 0)
+    (property "Reference" "C34" (id 0) (at 467.36 153.67 0)
       (effects (font (size 1.27 1.27)) (justify left))
     )
-    (property "Value" "47pF" (id 1) (at 482.6 168.91 0)
+    (property "Value" "47pF" (id 1) (at 467.36 157.48 0)
       (effects (font (size 1.27 1.27)) (justify left))
     )
-    (property "Footprint" "CAPC1608X90" (id 2) (at 478.79 170.18 0)
+    (property "Footprint" "CAPC1608X90" (id 2) (at 471.17 157.48 0)
       (effects (font (size 1.27 1.27)) (justify left bottom) hide)
     )
-    (property "Datasheet" "" (id 3) (at 478.79 170.18 0)
+    (property "Datasheet" "" (id 3) (at 471.17 157.48 0)
       (effects (font (size 1.27 1.27)) (justify left bottom) hide)
     )
@@
       (effects (font (size 1.27 1.27)) (justify left))
     )
-    (property "Value" "47pF" (id 1) (at 461.01 158.75 0)
+    (property "Value" "47pF" (id 1) (at 461.01 157.48 0)
       (effects (font (size 1.27 1.27)) (justify left))
     )
@@
       (effects (font (size 1.27 1.27)) (justify left))
     )
-    (property "Value" "100n" (id 1) (at 407.67 156.21 0)
+    (property "Value" "100n" (id 1) (at 405.13 154.94 0)
       (effects (font (size 1.27 1.27)) (justify left))
     )
@@
     (pin "1")
   )
-  (symbol (lib_id "power:GND") (at 478.79 172.72 0) (mirror y) (unit 1)
+  (symbol (lib_id "power:GND") (at 471.17 154.94 0) (mirror x) (unit 1)
     (in_bom yes) (on_board yes)
-    (property "Reference" "#PWR0115" (id 0) (at 478.79 179.07 0)
+    (property "Reference" "#PWR0115" (id 0) (at 471.17 148.59 0)
       (effects (font (size 1.27 1.27)) hide)
     )
-    (property "Value" "GND" (id 1) (at 474.98 173.99 0))
-    (property "Footprint" "" (id 2) (at 478.79 172.72 0)
+    (property "Value" "GND" (id 1) (at 474.98 153.67 0))
+    (property "Footprint" "" (id 2) (at 471.17 154.94 0)
       (effects (font (size 1.27 1.27)) hide)
     )
-    (property "Datasheet" "" (id 3) (at 478.79 172.72 0)
+    (property "Datasheet" "" (id 3) (at 471.17 154.94 0)
       (effects (font (size 1.27 1.27)) hide)
     )

Commit message: Update capacitors in microcontroller block
Parts:
- removed C13, C14, C15, C16, C17, C18, C19, C22: 100n, CAPC1608X90, symbol STM32_Breakout-rescue:CC0603MRX5R5BB475-CC0603MRX5R5BB475
- C12: value 100n -> 1u
Connections:
- net +3V3: no longer U4.108 (VDD), U4.121 (VDD), U4.144 (VDD), U4.17 (VDD), U4.39 (VDD), U4.52 (VDD), U4.62 (VDD), U4.72 (VDD), U4.84 (VDD)
- net VDDMAIN: now reaches C10.2, C12.2, D5.2 (A), FB5.1
- net VDDMAIN: now also U4.108 (VDD), U4.121 (VDD), U4.144 (VDD), U4.17 (VDD), U4.39 (VDD), U4.52 (VDD), U4.62 (VDD), U4.72 (VDD), U4.84 (VDD)

Commit message: Layout Adjustments
Connections:
- net I2C1-SCL is gone; now on net I2C1_SCL: U4.129 (PG14)
- net I2C1-SDA is gone; now on net I2C1_SDA: U4.128 (PG13)
- net SP1_NSS is gone; now on net SPI1_NSS: U6.1 (CS)
- net SPI2_CLK is gone; now on net SPI2_SCK: J7.5, U4.69 (PB10)
- net SPI1_MISO: now also U4.88 (PG3)
- net SPI1_MOSI: now also U4.89 (PG4)
- net SPI1_SCK: now also U4.87 (PG2)
- net SPI1_NSS: now reaches U4.65 (PE12)
Changed lines of the file:
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@@
     )
   )
-  (global_label "SPI2_CLK" (shape input) (at 430.53 312.42 180) (fields_autoplaced)
-    (effects (font (size 1.27 1.27)) (justify right))
-    (property "Intersheet References" "${INTERSHEET_REFS}" (id 0) (at 0 0 0)
-      (effects (font (size 1.27 1.27)) hide)
+  (global_label "SPI2_SCK" (shape input) (at 430.53 312.42 180) (fields_autoplaced)
+    (effects (font (size 1.27 1.27)) (justify right))
+    (property "Intersheet References" "${INTERSHEET_REFS}" (id 0) (at 419.1948 312.3406 0)
+      (effects (font (size 1.27 1.27)) (justify right) hide)
     )
   )
@@
     )
   )
+  (global_label "SPI1_NSS" (shape input) (at 262.89 280.67 180) (fields_autoplaced)
+    (effects (font (size 1.27 1.27)) (justify right))
+    (property "Intersheet References" "${INTERSHEET_REFS}" (id 0) (at 251.5548 280.5906 0)
+      (effects (font (size 1.27 1.27)) (justify right) hide)
+    )
+  )
+  (global_label "SPI1_MISO" (shape input) (at 328.93 257.81 0) (fields_autoplaced)
+    (effects (font (size 1.27 1.27)) (justify left))
+    (property "Intersheet References" "${INTERSHEET_REFS}" (id 0) (at 341.1118 257.7306 0)
+      (effects (font (size 1.27 1.27)) (justify left) hide)
+    )
+  )
   (global_label "VDDIO2" (shape input) (at 322.58 97.79 0) (fields_autoplaced)
     (effects (font (size 1.27 1.27)) (justify left))
@@
     )
   )
-  (global_label "I2C1-SDA" (shape input) (at 328.93 283.21 0) (fields_autoplaced)
-    (effects (font (size 1.27 1.27)) (justify left))
-    (property "Intersheet References" "${INTERSHEET_REFS}" (id 0) (at 0 0 0)
-      (effects (font (size 1.27 1.27)) hide)
+  (global_label "I2C1_SDA" (shape input) (at 328.93 283.21 0) (fields_autoplaced)
+    (effects (font (size 1.27 1.27)) (justify left))
+    (property "Intersheet References" "${INTERSHEET_REFS}" (id 0) (at 340.0837 283.1306 0)
+      (effects (font (size 1.27 1.27)) (justify left) hide)
     )
   )
@@
     )
   )
+  (global_label "SPI1_MOSI" (shape input) (at 328.93 260.35 0) (fields_autoplaced)
+    (effects (font (size 1.27 1.27)) (justify left))
+    (property "Intersheet References" "${INTERSHEET_REFS}" (id 0) (at 341.1118 260.2706 0)
+      (effects (font (size 1.27 1.27)) (justify left) hide)
+    )
+  )
   (global_label "SPI2_MISO" (shape input) (at 416.56 87.63 0) (fields_autoplaced)
     (effects (font (size 1.27 1.27)) (justify left))
@@
     )
   )
-  (global_label "I2C1-SCL" (shape input) (at 328.93 285.75 0) (fields_autoplaced)
-    (effects (font (size 1.27 1.27)) (justify left))
-    (property "Intersheet References" "${INTERSHEET_REFS}" (id 0) (at 0 0 0)
-      (effects (font (size 1.27 1.27)) hide)
+  (global_label "I2C1_SCL" (shape input) (at 328.93 285.75 0) (fields_autoplaced)
+    (effects (font (size 1.27 1.27)) (justify left))
+    (property "Intersheet References" "${INTERSHEET_REFS}" (id 0) (at 340.0232 285.6706 0)
+      (effects (font (size 1.27 1.27)) (justify left) hide)
     )
   )
@@
     )
   )
-  (global_label "SP1_NSS" (shape input) (at 450.85 246.38 270) (fields_autoplaced)
-    (effects (font (size 1.27 1.27)) (justify right))
-    (property "Intersheet References" "${INTERSHEET_REFS}" (id 0) (at 0 0 0)
-      (effects (font (size 1.27 1.27)) hide)
+  (global_label "SPI1_NSS" (shape input) (at 450.85 246.38 270) (fields_autoplaced)
+    (effects (font (size 1.27 1.27)) (justify right))
+    (property "Intersheet References" "${INTERSHEET_REFS}" (id 0) (at 450.7706 257.7152 90)
+      (effects (font (size 1.27 1.27)) (justify right) hide)
     )
   )
@@
     )
   )
-  (global_label "SPI2_CLK" (shape input) (at 265.43 209.55 180) (fields_autoplaced)
-    (effects (font (size 1.27 1.27)) (justify right))
-    (property "Intersheet References" "${INTERSHEET_REFS}" (id 0) (at 0 0 0)
-      (effects (font (size 1.27 1.27)) hide)
+  (global_label "SPI2_SCK" (shape input) (at 265.43 209.55 180) (fields_autoplaced)
+    (effects (font (size 1.27 1.27)) (justify right))
+    (property "Intersheet References" "${INTERSHEET_REFS}" (id 0) (at 254.0948 209.4706 0)
+      (effects (font (size 1.27 1.27)) (justify right) hide)
     )
   )
@@
     )
   )
+  (global_label "SPI1_SCK" (shape input) (at 328.93 255.27 0) (fields_autoplaced)
+    (effects (font (size 1.27 1.27)) (justify left))
+    (property "Intersheet References" "${INTERSHEET_REFS}" (id 0) (at 340.2652 255.1906 0)
+      (effects (font (size 1.27 1.27)) (justify left) hide)
+    )
+  )
