File: OBC_Boards/5V to 3V3/qsat5to3.3.sch (KiCad schematic (older format))
At the start: 6 parts

Commit message: Add clock circuitry and power circuitry. Add footprints for devices that did not have any. Add ferrite beads as inputs to each power source for each circuit
Parts:
- D?: footprint (none) -> Package_TO_SOT_SMD:SOT-23
- U?: symbol qsat-symb:BU33SA5WGWZ-E2 -> qsat5to3.3-rescue:BU33SA5WGWZ-E2-qsat-symb
Changed lines of the file:
@@
 EESchema Schematic File Version 4
+LIBS:qsat5to3.3-cache
 EELAYER 30 0
 EELAYER END
@@
 $EndDescr
 $Comp
-L qsat-symb:BU33SA5WGWZ-E2 U?
+L qsat5to3.3-rescue:BU33SA5WGWZ-E2-qsat-symb U?
 U 1 1 617B1000
 P 7500 2300
@@
 F 0 "D?" V 6104 3180 50  0000 L CNN
 F 1 "10V" V 6195 3180 50  0000 L CNN
-F 2 "" H 6150 3100 50  0001 C CNN
+F 2 "Package_TO_SOT_SMD:SOT-23" H 6150 3100 50  0001 C CNN
 F 3 "~" H 6150 3100 50  0001 C CNN
 	1    6150 3100
