File: OBC_Boards/DebugBoard/_autosave-DebugBoard.kicad_sch (KiCad schematic)
At the start: 16 parts, among them J1 Conn_01x02_Female, J2 Conn_02x06_Counter_Clockwise, J3 Conn_01x03, P1 USB_C_Plug_USB2.0, U1 L102021MS02Q

Commit message: dev
Parts:
- removed TP4: TestPoint, symbol Connector:TestPoint
- TP2, TP3: footprint (none) -> TestPoint:TestPoint_Pad_2.0x2.0mm
Connections:
- net 5V Input is gone; now on net 5V0_IN: U1.3
- net VCC_3V3 is gone; now on net 3V3_OUT: J1.1 (Pin_1)
- net 3V3_OUT: now also TP1.1
- net 5V0-CHG: now also U1.1; no longer U1.2
- net 5V0_IN: now also TP2.1
- net 5VUSB: now also U1.2; no longer U1.1
- net GND: now also TP3.1
Changed lines of the file:
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@@
     (stroke (width 0) (type default) (color 0 0 0 0))
   )
-  (polyline (pts (xy 157.48 53.34) (xy 157.48 85.09))
+  (polyline (pts (xy 152.4 53.34) (xy 152.4 85.09))
     (stroke (width 0) (type default) (color 0 0 0 0))
   )
@@
     (stroke (width 0) (type default) (color 0 0 0 0))
   )
-  (polyline (pts (xy 157.48 53.34) (xy 190.5 53.34))
+  (polyline (pts (xy 152.4 53.34) (xy 190.5 53.34))
     (stroke (width 0) (type default) (color 0 0 0 0))
   )
@@
     (stroke (width 0) (type default) (color 0 0 0 0))
   )
-  (polyline (pts (xy 190.5 85.09) (xy 157.48 85.09))
+  (polyline (pts (xy 190.5 85.09) (xy 152.4 85.09))
     (stroke (width 0) (type default) (color 0 0 0 0))
   )
@@
     )
   )
-  (global_label "VCC_3V3" (shape output) (at 167.64 142.24 180) (fields_autoplaced)
+  (global_label "3V3_OUT" (shape output) (at 167.64 142.24 180) (fields_autoplaced)
     (effects (font (size 1.27 1.27)) (justify right))
     (property "Intersheet References" "${INTERSHEET_REFS}" (id 0) (at 157.1231 142.1606 0)
@@
     )
   )
-  (global_label "5VUSB" (shape input) (at 127 107.95 180) (fields_autoplaced)
-    (effects (font (size 1.27 1.27)) (justify right))
-    (property "Intersheet References" "${INTERSHEET_REFS}" (id 0) (at 118.4788 107.8706 0)
-      (effects (font (size 1.27 1.27)) (justify right) hide)
+  (global_label "5VUSB" (shape output) (at 167.64 110.49 0) (fields_autoplaced)
+    (effects (font (size 1.27 1.27)) (justify left))
+    (property "Intersheet References" "${INTERSHEET_REFS}" (id 0) (at 176.1612 110.4106 0)
+      (effects (font (size 1.27 1.27)) (justify left) hide)
     )
   )
@@
     )
   )
-  (global_label "5V0-CHG" (shape output) (at 167.64 110.49 0) (fields_autoplaced)
-    (effects (font (size 1.27 1.27)) (justify left))
-    (property "Intersheet References" "${INTERSHEET_REFS}" (id 0) (at 179.0036 110.4106 0)
-      (effects (font (size 1.27 1.27)) (justify left) hide)
+  (global_label "5V0-CHG" (shape input) (at 127 107.95 180) (fields_autoplaced)
+    (effects (font (size 1.27 1.27)) (justify right))
+    (property "Intersheet References" "${INTERSHEET_REFS}" (id 0) (at 115.6364 107.8706 0)
+      (effects (font (size 1.27 1.27)) (justify right) hide)
     )
   )
@@
     )
   )
+  (global_label "5V0_IN" (shape output) (at 163.83 71.12 180) (fields_autoplaced)
+    (effects (font (size 1.27 1.27)) (justify right))
+    (property "Intersheet References" "${INTERSHEET_REFS}" (id 0) (at 155.0064 71.1994 0)
+      (effects (font (size 1.27 1.27)) (justify right) hide)
+    )
+  )
   (global_label "3V3_OUT" (shape output) (at 114.3 64.77 180) (fields_autoplaced)
     (effects (font (size 1.27 1.27)) (justify right))
@@
     )
   )
+  (global_label "5V0_IN" (shape output) (at 167.64 107.95 0) (fields_autoplaced)
+    (effects (font (size 1.27 1.27)) (justify left))
+    (property "Intersheet References" "${INTERSHEET_REFS}" (id 0) (at 176.4636 107.8706 0)
+      (effects (font (size 1.27 1.27)) (justify left) hide)
+    )
+  )
   (global_label "GND-CHG" (shape input) (at 127 62.23 0) (fields_autoplaced)
     (effects (font (size 1.27 1.27)) (justify left))
@@
     )
   )
-  (global_label "5V Input" (shape output) (at 167.64 107.95 0) (fields_autoplaced)
-    (effects (font (size 1.27 1.27)) (justify left))
-    (property "Intersheet References" "${INTERSHEET_REFS}" (id 0) (at 178.0964 107.8706 0)
-      (effects (font (size 1.27 1.27)) (justify left) hide)
+  (global_label "3V3_OUT" (shape output) (at 163.83 63.5 180) (fields_autoplaced)
+    (effects (font (size 1.27 1.27)) (justify right))
+    (property "Intersheet References" "${INTERSHEET_REFS}" (id 0) (at 153.3131 63.4206 0)
+      (effects (font (size 1.27 1.27)) (justify right) hide)
     )
   )
@@
     (pin "1")
   )
-  (symbol (lib_id "Connector:TestPoint") (at 163.83 82.55 0) (unit 1)
-    (in_bom yes) (on_board yes) (fields_autoplaced)
-    (property "Reference" "TP4" (id 0) (at 166.37 77.9779 0)
-      (effects (font (size 1.27 1.27)) (justify left))
-    )
-    (property "Value" "TestPoint" (id 1) (at 166.37 80.5179 0)
-      (effects (font (size 1.27 1.27)) (justify left))
-    )
-    (property "Footprint" "" (id 2) (at 168.91 82.55 0)
-      (effects (font (size 1.27 1.27)) hide)
-    )
-    (property "Datasheet" "~" (id 3) (at 168.91 82.55 0)
-      (effects (font (size 1.27 1.27)) hide)
-    )
-    (pin "1")
-  )
   (symbol (lib_id "Device:LED") (at 60.96 63.5 90) (unit 1)
     (in_bom yes) (on_board yes) (fields_autoplaced)
@@
     (pin "1")
     (pin "2")
-  )
-  (symbol (lib_id "Connector:TestPoint") (at 163.83 69.85 0) (unit 1)
-    (in_bom yes) (on_board yes) (fields_autoplaced)
-    (property "Reference" "TP2" (id 0) (at 166.37 65.2779 0)
-      (effects (font (size 1.27 1.27)) (justify left))
-    )
-    (property "Value" "TestPoint" (id 1) (at 166.37 67.8179 0)
-      (effects (font (size 1.27 1.27)) (justify left))
-    )
-    (property "Footprint" "" (id 2) (at 168.91 69.85 0)
-      (effects (font (size 1.27 1.27)) hide)
-    )
-    (property "Datasheet" "~" (id 3) (at 168.91 69.85 0)
-      (effects (font (size 1.27 1.27)) hide)
-    )
-    (pin "1")
   )
   (symbol (lib_id "Device:R") (at 72.39 76.2 0) (unit 1)
@@
     (pin "1")
   )
+  (symbol (lib_id "Connector:TestPoint") (at 163.83 71.12 0) (unit 1)
+    (in_bom yes) (on_board yes) (fields_autoplaced)
+    (property "Reference" "TP2" (id 0) (at 166.37 66.5479 0)
+      (effects (font (size 1.27 1.27)) (justify left))
+    )
+    (property "Value" "TestPoint" (id 1) (at 166.37 69.0879 0)
+      (effects (font (size 1.27 1.27)) (justify left))
+    )
+    (property "Footprint" "TestPoint:TestPoint_Pad_2.0x2.0mm" (id 2) (at 168.91 71.12 0)
+      (effects (font (size 1.27 1.27)) hide)
+    )
+    (property "Datasheet" "~" (id 3) (at 168.91 71.12 0)
+      (effects (font (size 1.27 1.27)) hide)
+    )
+    (pin "1")
+  )
   (symbol (lib_id "Device:LED") (at 83.82 63.5 90) (unit 1)
     (in_bom yes) (on_board yes) (fields_autoplaced)
@@
     (pin "9")
   )
-  (symbol (lib_id "Connector:TestPoint") (at 163.83 76.2 0) (unit 1)
-    (in_bom yes) (on_board yes) (fields_autoplaced)
-    (property "Reference" "TP3" (id 0) (at 166.37 71.6279 0)
-      (effects (font (size 1.27 1.27)) (justify left))
-    )
-    (property "Value" "TestPoint" (id 1) (at 166.37 74.1679 0)
-      (effects (font (size 1.27 1.27)) (justify left))
-    )
-    (property "Footprint" "" (id 2) (at 168.91 76.2 0)
-      (effects (font (size 1.27 1.27)) hide)
-    )
-    (property "Datasheet" "~" (id 3) (at 168.91 76.2 0)
-      (effects (font (size 1.27 1.27)) hide)
-    )
-    (pin "1")
-  )
   (symbol (lib_id "Daughterboard_Symbols:L102021MS02Q") (at 127 107.95 0) (unit 1)
     (in_bom yes) (on_board yes) (fields_autoplaced)
@@
     (pin "1")
   )
+  (symbol (lib_id "Connector:TestPoint") (at 163.83 80.01 0) (unit 1)
+    (in_bom yes) (on_board yes) (fields_autoplaced)
+    (property "Reference" "TP3" (id 0) (at 166.37 75.4379 0)
+      (effects (font (size 1.27 1.27)) (justify left))
+    )
+    (property "Value" "TestPoint" (id 1) (at 166.37 77.9779 0)
+      (effects (font (size 1.27 1.27)) (justify left))
+    )
+    (property "Footprint" "TestPoint:TestPoint_Pad_2.0x2.0mm" (id 2) (at 168.91 80.01 0)
+      (effects (font (size 1.27 1.27)) hide)
+    )
+    (property "Datasheet" "~" (id 3) (at 168.91 80.01 0)
+      (effects (font (size 1.27 1.27)) hide)
+    )
+    (pin "1")
+  )
   (symbol (lib_id "power:GND") (at 114.3 67.31 270) (unit 1)
     (in_bom yes) (on_board yes) (fields_autoplaced)
@@
     )
     (property "Datasheet" "" (id 3) (at 114.3 67.31 0)
+      (effects (font (size 1.27 1.27)) hide)
+    )
+    (pin "1")
+  )
+  (symbol (lib_id "power:GND") (at 163.83 80.01 0) (unit 1)
+    (in_bom yes) (on_board yes)
+    (property "Reference" "#PWR09" (id 0) (at 163.83 86.36 0)
+      (effects (font (size 1.27 1.27)) hide)
+    )
+    (property "Value" "GND" (id 1) (at 160.02 82.55 0))
+    (property "Footprint" "" (id 2) (at 163.83 80.01 0)
+      (effects (font (size 1.27 1.27)) hide)
+    )
+    (property "Datasheet" "" (id 3) (at 163.83 80.01 0)
       (effects (font (size 1.27 1.27)) hide)
     )
@@
       (reference "#PWR08") (unit 1) (value "GND") (footprint "")
     )
+    (path "/f1bc33b1-d1c6-47f4-ac16-d213fa0e3867"
+      (reference "#PWR09") (unit 1) (value "GND") (footprint "")
+    )
     (path "/c97d4d8f-67f5-43c7-8ee8-cf68b574a8f6"
       (reference "#PWR0101") (unit 1) (value "GND") (footprint "")
@@
       (reference "TP1") (unit 1) (value "TestPoint") (footprint "")
     )
-    (path "/2f890fd3-8730-4355-9587-698a6082111b"
-      (reference "TP2") (unit 1) (value "TestPoint") (footprint "")
-    )
-    (path "/c591f571-37ab-4639-94a5-281cb4e19198"
-      (reference "TP3") (unit 1) (value "TestPoint") (footprint "")
-    )
-    (path "/04962a07-cc1b-4504-a8bc-3dd2947448cc"
-      (reference "TP4") (unit 1) (value "TestPoint") (footprint "")
+    (path "/a0395d07-65f8-4c65-a9d0-f3e64c260792"
+      (reference "TP2") (unit 1) (value "TestPoint") (footprint "TestPoint:TestPoint_Pad_2.0x2.0mm")
+    )
+    (path "/d971024d-e6bc-4b36-8c60-4cb62daf9b6d"
+      (reference "TP3") (unit 1) (value "TestPoint") (footprint "TestPoint:TestPoint_Pad_2.0x2.0mm")
     )
     (path "/c69eb4af-e3dc-4ec4-b995-490bbddceacb"
