File: OBC_Boards/DebugBoard/DebugBoard.kicad_pcb (KiCad board)
At the start: 4 copper layers, 45.1 x 43.2 mm, 19 parts, among them J1 Conn_01x02_Female, J2 Conn_02x06_Counter_Clockwise, J3 Conn_01x03, P1 USB_C_Plug_USB2.0, U1 S1

Commit message: OBC: umb-db: generate manufacturing files for ordering
Parts:
- removed 3V3, 5V0, GND: TestPoint, TestPoint:TestPoint_Pad_2.0x2.0mm
- added G***: LOGO, LOGO, F.Cu at (124.8, 79.3)
- added TP1: 3V3, TestPoint:TestPoint_Pad_2.0x2.0mm, F.Cu at (106.3, 115.1)
- added TP2: 5V0, TestPoint:TestPoint_Pad_2.0x2.0mm, F.Cu at (109.8, 115.1)
- added TP3: GND, TestPoint:TestPoint_Pad_2.0x2.0mm, F.Cu at (113.3, 115.1)
- U1: value S1 -> L102021MS02Q; footprint Daughterboard_footprints:L102021MS02Q -> qset-footprints:L102021MS02Q
- moved J3 5.75 mm to (132.7, 82.6)
- moved BZ1 3.35 mm to (122.9, 93.1)
Routing:
- net 3V3_OUT: track 56.5 -> 5.01 mm, vias 0 -> 3
- net 5V0_IN: track 56.3 -> 18.4 mm, vias 2 -> 1
- net I2C_SDA: track 44.9 -> 36.9 mm
- net GND: track 11.8 -> 3.84 mm, vias 1 -> 2
- net I2C_SDK: track 53.4 -> 47.9 mm
- net Buzzer/GPIO_1: track 25.0 -> 22.2 mm
- added copper zone on In2.Cu, net 3V3_OUT
Other:
- board text added: "2022-2023"
- board text added: "SN:______"
- board text added: "Umbilical Debug Board"
