File: ADCS_Boards/MC_SunSensorPCB/MC_SunSensorPCB.kicad_sch (KiCad schematic)
At the start: 66 parts, among them J1 PC104_Connector, U1 CM9V-T1A, U10 Op-Amp, U11 Op-Amp, U12 Op-Amp, U13 Op-Amp, U2 MCP7940NT-I_MS, U3 MR25H10MDF, U4 DF13-4P-1.25DS(20), U5 DF13-4P-1.25DS(20), U6 DF13-4P-1.25DS(20), U7 DF13-4P-1.25DS(20), U8 LM358, U9 CD74HC4067M96

Commit message: Updated RW and MCU PCBS. Layouts are complete, just need to do routing. (Pushed for Yasin Shahrami)
Parts:
- removed BT1: Battery_Cell, symbol Device:Battery_Cell
- removed C1: 100n, CAPC1608X90, symbol STM32_Breakout-rescue:CC0603MRX5R5BB475-CC0603MRX5R5BB475
- removed D1: RED, LED_SMD:LED_0603_1608Metric_Pad1.05x0.95mm_HandSolder, symbol Device:LED_Small
- removed R1, R2, R3: 10k, symbol Device:R
- removed R4: 2k2, RESC1607X60N, symbol STM32_Breakout-rescue:R0603-OBC_Libary
- removed R5, R6: 10k, RESC1607X60N, symbol STM32_Breakout-rescue:R0603-OBC_Libary
- removed U1: CM9V-T1A, symbol qsat-symb:CM9V-T1A
- removed U2: MCP7940NT-I_MS, symbol qsat-symb:MCP7940NT-I_MS
- removed U3: MR25H10MDF, STM32_Breakout:SON65P300X300X95-8N, symbol STM32_Breakout-rescue:MR25H10MDF-MRAM_Symbol
- removed U4, U5, U6, U7: DF13-4P-1.25DS(20), Footprints_QSAT:DF13-6P-1.25DS(20), symbol DF13_Connector:DF13-4P-1.25DS(20)
- added C1, C24, C27, C30: 1.0uF, SparkFun_IMU_Breakout_ICM-20948:0603, symbol SparkFun_IMU_Breakout_ICM-20948-eagle-import:1.0UF-0603-16V-10%-X7R
- added C22, C23, C28, C29: 0.1uF, SparkFun_IMU_Breakout_ICM-20948:0603, symbol SparkFun_IMU_Breakout_ICM-20948-eagle-import:0.1UF-0603-25V-5%
- added C25, C26: 10p, Capacitor_SMD:C_0603_1608Metric, symbol Device:C
- added C31: 100n, STM32_Breakout:CAPC1608X90, symbol STM32_Breakout-rescue:CC0603MRX5R5BB475-CC0603MRX5R5BB475
- added D1, D2: RED, SparkFun_IMU_Breakout_ICM-20948:LED-0603, symbol SparkFun_IMU_Breakout_ICM-20948-eagle-import:LED-RED0603
- added D3: RED, LED_SMD:LED_0603_1608Metric_Pad1.05x0.95mm_HandSolder, symbol Device:LED_Small
- added J2: PPTC062LJBN-RC, Footprints_QSAT:PPTC062LJBN-RC, symbol ADCS_Symbols:PPTC062LJBN-RC
- added J3: Conn_01x03_Female, Footprints_QSAT:1x3_Connector_Female, symbol Connector:Conn_01x03_Female
- added JP2, JP5: I2C PU, SparkFun_IMU_Breakout_ICM-20948:SMT-JUMPER_3_2-NC_TRACE_SILK, symbol SparkFun_IMU_Breakout_ICM-20948-eagle-import:JUMPER-SMT_3_2-NC_TRACE_SILK
- added JP3, JP6: LED, SparkFun_IMU_Breakout_ICM-20948:SMT-JUMPER_2_NC_TRACE_SILK, symbol SparkFun_IMU_Breakout_ICM-20948-eagle-import:JUMPER-SMT_2_NC_TRACE_SILK
- added Q12, Q14, Q3, Q4, Q6, Q9: 20V/0.2A/8MHz/1.2Ω/1Vth, SparkFun_IMU_Breakout_ICM-20948:SOT-416FL, symbol SparkFun_IMU_Breakout_ICM-20948-eagle-import:MOSFET-NCH-RE1C002UN
- added R1, R26, R27, R28, R29, R3, R32, R33, R40, R43, R46, R47: 2.2k, SparkFun_IMU_Breakout_ICM-20948:0402-TIGHT, symbol SparkFun_IMU_Breakout_ICM-20948-eagle-import:2.2KOHM-0402T-1/16W-1%
- added R36, R51: 220, SparkFun_IMU_Breakout_ICM-20948:0603, symbol SparkFun_IMU_Breakout_ICM-20948-eagle-import:220OHM-0603-1/10W-1%
- added R53: 2k2, STM32_Breakout:RESC1607X60N, symbol STM32_Breakout-rescue:R0603-OBC_Libary
- added R54, R55: 10k, STM32_Breakout:RESC1607X60N, symbol STM32_Breakout-rescue:R0603-OBC_Libary
- added TP1, TP2: 1.8V, SparkFun_IMU_Breakout_ICM-20948:PAD.03X.03, symbol SparkFun_IMU_Breakout_ICM-20948-eagle-import:TEST-POINT3
- added U1, U3: 9DoF IMU, SparkFun_IMU_Breakout_ICM-20948:QFN24-3X3, symbol SparkFun_IMU_Breakout_ICM-20948-eagle-import:ICM-20948
- added U14, U2: 1.8V/100mA, SparkFun_IMU_Breakout_ICM-20948:SC70, symbol SparkFun_IMU_Breakout_ICM-20948-eagle-import:V_REG_SP6214-1.8V
- added U15: STM32F103RET6, Footprints_QSAT:QFP50P1200X1200X160-64N, symbol ADCS_Symbols:STM32F103RET6
- added U16: MR25H10MDF, STM32_Breakout:SON65P300X300X95-8N, symbol STM32_Breakout-rescue:MR25H10MDF-MRAM_Symbol
- added U4, U5, U6, U7: DF13-7P-1.25DS(20), Connector_Hirose:Hirose_DF13-07P-1.25DS_1x07_P1.25mm_Horizontal, symbol ADCS_Symbols:DF13-4P-1.25DS(20)
- added Y1: Crystal_GND24, Crystal:Crystal_SMD_3225-4Pin_3.2x2.5mm, symbol Device:Crystal_GND24
- C10, C11, C12, C13, C14, C15, C16, C17, C18, C19, C2, C20, C21, C3, C4, C5, C6, C7, C8, C9: footprint Capacitor_THT:CP_Radial_D4.0mm_P2.00mm -> Capacitor_SMD:C_0603_1608Metric
- R10, R11, R12, R13, R14, R15, R16, R17, R18, R19, R20, R21, R22, R23, R24, R7, R8, R9: footprint Resistor_THT:R_Axial_DIN0204_L3.6mm_D1.6mm_P1.90mm_Vertical -> Resistor_SMD:R_0603_1608Metric
Connections:
- net 3V3 is gone; now on net +3V3: FB1.1, J1.79 (H2-27)
- net +3V3: now also R54.2, R55.2, U15.32 (VDD_1)
- net GND: now also J1.100 (H2-48), J1.99 (H2-47), C1.2, C22.2, C23.2, C24.2, C25.2, C26.2, C27.2, C28.2, C29.2, C30.2, C31.1, JP3.1, JP6.1, R53.2, U1.18 (GND), U1.20 (GND), U14.2 (GND), U15.31 (VSS_1), U16.4 (VSS), U16.9 (Sink), U2.2 (GND), U3.18 (GND), U3.20 (GND), U4.2, U4.4, U4.6, U5.2, U5.4, U5.6, U6.2, U6.4, U6.6, U7.2, U7.4, U7.6, Y1.2, Y1.4
- net MuxEnable: now also U15.14 (PA0-WKUP/USART2_CTS/ADC123_IN0/TIM2_CH1_ETR/TIM5_CH1/TIM8_ETR); no longer J1.10 (H1-10)
- net MuxOut: now also U15.21 (PA5/SPI1_SCK/DAC_OUT2/ADC12_IN5); no longer J1.15 (H1-15)
- net MuxS0: now also U15.15 (PA1/USART2_RTS/ADC123_IN1/TIM5_CH2/TIM2_CH2); no longer J1.11 (H1-11)
- net MuxS1: now also U15.16 (PA2/USART2_TX/TIM5_CH3/ADC123_IN2/TIM2_CH3); no longer J1.12 (H1-12)
- net MuxS2: now also U15.17 (PA3/USART2_RX/TIM5_CH4/ADC123_IN3/TIM2_CH4); no longer J1.13 (H1-13)
- net MuxS3: now also U15.20 (PA4/SPI1_NSS/USART2_CK/DAC_OUT1/ADC12_IN4); no longer J1.14 (H1-14)
- net PD1_O1: now also U5.1
- net PD1_O2: now also U4.1
- net PD1_O3: now also U6.1
- net PD1_O4: now also U7.1
- net PD2_O1: now also U5.3
- net PD2_O2: now also U4.3
- net PD2_O3: now also U6.3
- net PD2_O4: now also U7.3
- net PD3_O1: now also U5.5
- net PD3_O2: now also U4.5
- net PD3_O3: now also U6.5
- net PD3_O4: now also U7.5
- net PD4_O1: now also U5.7
- net PD4_O2: now also U4.7
- net PD4_O3: now also U6.7
- net PD4_O4: now also U7.7
- net SPI1_MISO: now also U15.11 (PC3/ADC123_IN13), U16.2 (SO)
- net SPI1_MOSI: now also U15.9 (PC1/ADC123_IN11), U16.5 (SI)
- net SPI1_NSS: now also U15.10 (PC2/ADC123_IN12), U16.1 (CS)
- net SPI1_SCK: now also U15.8 (PC0/ADC123_IN10), U16.6 (SCK)
- net at FB1.2: now also C31.2, D3.2 (A), U16.8 (VDD)
- net PA6: now reaches J1.16 (H1-16)
- net PA6: now also U15.22 (PA6/SPI1_MISO/TIM8_BKIN/ADC12_IN6/TIM3_CH1)
- net PA7: now reaches J1.17 (H1-17)
- net PA7: now also U15.23 (PA7/SPI1_MOSI/TIM8_CH1N/ADC12_IN7/TIM3_CH2)
- net PA8: now reaches J1.18 (H1-18)
- net PA8: now also U15.41 (PA8/USART1_CK/TIM1_CH1/MCO)
- net PA9: now reaches J1.19 (H1-19)
- net PA9: now also U15.42 (PA9/USART1_TX/TIM1_CH2)
- net PA10: now reaches J1.20 (H1-20)
- net PA10: now also U15.43 (PA10/USART1_RX/TIM1_CH3)
- net PA11: now reaches J1.21 (H1-21)
- net PA11: now also U15.44 (PA11/USART1_CTS/USBDMCAN_RX/TIM1_CH4)
- net PA12: now reaches J1.22 (H1-22)
- net PA12: now also U15.45 (PA12/USART1_RTS/USBDP/CAN_TX/TIM1_ETR)
- net PB10: now reaches J1.23 (H1-23)
- net PB10: now also U15.29 (PB10/I2C2_SCL/USART3_TX/TIM2_CH3)
- net PB0: now reaches J1.24 (H1-24)
- net PB0: now also U15.26 (PB0/ADC12_IN8/TIM3_CH3/TIM8_CH2N)
- net PA15: now reaches J1.25 (H1-25)
- net PA15: now also U15.50 (PA15/SPI3_NSS/I2S3_WS)
- net PB12: now reaches J1.26 (H1-26)
- net PB12: now also U15.33 (PB12/SPI2_NSS/I2S2_WS/I2C2_SMBA/USART3_CK/TIM1_BKIN)
- net PB13: now reaches J1.27 (H1-27)
- net PB13: now also U15.34 (PB13/SPI2_SCK/I2S2_CK/USART3_CTS/TIM1_CH1N)
- net PB14: now reaches J1.37 (H1-37)
- net PB14: now also U15.35 (PB14/SPI2_MISO/TIM1_CH2N/USART3_RTS)
- net PB15: now reaches J1.38 (H1-38)
- net PB15: now also U15.36 (PB15/SPI2_MOSI/I2S2_SD/TIM1_CH3N)
- net PC6: now reaches J1.39 (H1-39)
- net PC6: now also U15.37 (PC6/I2S2_MCK/TIM8_CH1/SDIO_D6/TIM3_CH1)
- net PC7: now reaches J1.40 (H1-40)
- net PC7: now also U15.38 (PC7/I2S3_MCK/TIM8_CH2/SDIO_D7/TIM3_CH2)
- net at J1.41 (H1-41): now also J2.12, U15.59 (PB7/I2C1_SDA/FSMC_NADV/TIM4_CH2/USART1_RX)
- net PB1: now reaches J1.42 (H1-42)
- net PB1: now also U15.27 (PB1/ADC12_IN9/TIM3_CH4/TIM8_CH3N)
- net at J1.43 (H1-43): now also J2.11, U15.58 (PB6/I2C1_SCL/TIM4_CH1/USART1_TX)
- net PC11: now reaches J1.44 (H1-44)
- net PC11: now also U15.52 (PC11/UART4_RX/SDIO_D3/USART3_RX)
- net PC12: now reaches J1.45 (H1-45)
- net PC12: now also U15.53 (PC12/UART5_TX/SDIO_CK/USART3_CK)
- net PC13: now reaches J1.46 (H1-46)
- net PC13: now also U15.2 (PC13-TAMPER-RTC)
- net PC14: now reaches J1.47 (H1-47)
- net PC14: now also U15.3 (PC14-OSC32_IN)
- net PC15: now reaches J1.48 (H1-48)
- net PC15: now also U15.4 (PC15-OSC32_OUT)
- net PD2: now reaches J1.49 (H1-49)
- net PD2: now also U15.54 (PD2/TIM3_ETR/UART5_RX/SDIO_CMD)
- net PC10: now reaches J1.5 (H1-5)
- net PC10: now also U15.51 (PC10/UART4_TX/SDIO_D2/USART3_TX)
- net PB4: now reaches J1.50 (H1-50)
- net PB4: now also U15.56 (PB4/SPI3_MISO/TIM3_CH1/SPI1_MISO)
- net PB11: now reaches J1.51 (H1-51)
- net PB11: now also U15.30 (PB11/2C2_SDA/USART3_RX/TIM2_CH4)
- net PB8: now reaches J1.52 (H1-52)
- net PB8: now also U15.61 (PB8/TIM4_CH3/SDIO_D4/I2C1_SCL/CAN_RX)
- net 5V renamed +5V
- net +5V: now also C24.1, C30.1, JP2.2, JP5.2, R33.2, R47.2, U14.1 (IN), U14.3 (EN), U2.1 (IN), U2.3 (EN)
- new net: JP6.2, R51.1
- new net: D2.C, R51.2
- new net: C29.1, U1.10 (REGOUT)
- new net: JP2.3, R29.2
- new net: D3.1 (K), R53.1
- new net: JP2.1, R27.2
- new net: JP3.2, R36.1
- new net: D1.C, R36.2
- new net: JP5.1, R3.2
- new net: C23.1, U3.10 (REGOUT)
- new net: JP5.3, R43.2
- new net 1.8V: C1.1, C22.1, C27.1, C28.1, D1.A, D2.A, Q12.1 (G), Q14.1 (G), Q3.1 (G), Q4.1 (G), Q6.1 (G), Q9.1 (G), R1.2, R26.2, R28.2, R32.2, R40.2, R46.2, TP1.P$1 (1), TP2.P$1 (1), U1.13 (VDD), U1.8 (VDDIO), U14.5 (OUT), U2.5 (OUT), U3.13 (VDD), U3.8 (VDDIO)
- new net AD0/SDO: Q6.2 (S), R32.1, U15.28 (PB2//BOOT1), U3.9 (AD0/SDO)
- new net AD0/SDO_VIN: Q6.3 (D), R33.1
- new net AD0/SDO_2: Q14.2 (S), R46.1, U1.9 (AD0/SDO), U15.57 (PB5/TIM3_CH2/SPI1_MOSI/)
- new net AD0/SDO_VIN_2: Q14.3 (D), R47.1
- new net GPIO1: R54.1, U15.24 (PC4/ADC12_IN14), U16.7 (HOLD)
- new net GPIO2: R55.1, U15.25 (PC5/ADC12_IN15), U16.3 (WP)
- new net IMU_SCL: Q12.2 (S), Q4.2 (S), R28.1, R40.1, U1.23 (SCL/SCLK), U15.39 (PC8/TIM8_CH3/SDIO_D0/TIM3_CH3), U3.23 (SCL/SCLK)
- new net IMU_SDA: Q3.2 (S), Q9.2 (S), R1.1, R26.1, U1.24 (SDA/SDI), U15.40 (PC9/TIM8_CH4/SDIO_D1/TIM3_CH4), U3.24 (SDA/SDI)
- new net PB9: U15.62 (PB9/TIM4_CH4/SDIO_D5/I2C1_SDA/CAN_TX)
- new net RCC_OSC_IN: C25.1, U15.5 (PD0-OSC_IN/FSMC_D2/CAN_RX), Y1.1
- new net RCC_OSC_OUT: C26.1, U15.6 (PD1-OSC_OUT/FSMC_D3/CAN_TX), Y1.3
- new net SCL/SCLK_VIN: Q4.3 (D), R29.1
- new net SCL/SCLK_VIN_2: Q12.3 (D), R43.1
- new net SDA/SDI_VIN: Q3.3 (D), R27.1
- new net SDA/SDI_VIN_2: Q9.3 (D), R3.1
- new net SYS_JTCK-SWCLK: J3.2 (Pin_2), U15.49 (PA14/JTCKSWCLK)
- new net SYS_JTDO-TRACESWO: J3.3 (Pin_3), U15.55 (PB3/SPI3_SCK/I2S3_CK/TRACESWO/TIM2_CH2/SPI1_SCK)
- new net SYS_JTMS-SWDIO: J3.1 (Pin_1), U15.46 (PA13/JTMSSWDIO)
- no-connect marks 91 -> 76
Other:
- note added: "Cut to disable PWR LED"
- note added: "VIN 1.8V to 5.5V"
- moved on the sheet: C10, C11, C12, C13, C14, C15, C16, C17, C18, C19, C2, C20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
