File: comm-rfb/currentandvoltagemeasure.kicad_sch (KiCad schematic)
At the start: 0 parts

Commit message: added current monitor
Parts:
- added FB?: 100R @ 100 MHz, STM32_Breakout:INDUC1607X60N, symbol Device:Ferrite_Bead_Small
- added MAX4372F?: MAX4372FESA+, STM32_Breakout:SOIC127P600X175-8N, symbol STM32_Breakout-rescue:MAX4372FESA+-MAX4372FESA+
- added R?: 20m, RESC1607X60N, symbol STM32_Breakout-rescue:R0603-OBC_Libary
- added TP?: TestPoint, TestPoint:TestPoint_Pad_D2.0mm, symbol Connector:TestPoint
Connections:
- new net: FB?.1, MAX4372F?.1 (VCC)
- new net: MAX4372F?.8 (RS+), R?.1
- new net 3V3: FB?.2, MAX4372F?.6 (RS-), R?.2, TP?.1
- new net CURR-MONITOR: MAX4372F?.4 (OUT)
- new net GND: MAX4372F?.3 (GND)
Changed lines of the file:
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@@
 (kicad_sch (version 20211123) (generator eeschema)
   (paper "A4")
+  (junction (at 119.38 85.09) (diameter 0) (color 0 0 0 0)
+  )
+  (junction (at 116.84 82.55) (diameter 0) (color 0 0 0 0)
+  )
+  (wire (pts (xy 114.3 77.47) (xy 114.3 72.39))
+    (stroke (width 0) (type default) (color 0 0 0 0))
+  )
+  (wire (pts (xy 114.3 72.39) (xy 119.38 72.39))
+    (stroke (width 0) (type default) (color 0 0 0 0))
+  )
+  (wire (pts (xy 116.84 82.55) (xy 119.38 82.55))
+    (stroke (width 0) (type default) (color 0 0 0 0))
+  )
+  (wire (pts (xy 114.3 82.55) (xy 116.84 82.55))
+    (stroke (width 0) (type default) (color 0 0 0 0))
+  )
+  (wire (pts (xy 119.38 85.09) (xy 119.38 87.63))
+    (stroke (width 0) (type default) (color 0 0 0 0))
+  )
+  (wire (pts (xy 116.84 85.09) (xy 119.38 85.09))
+    (stroke (width 0) (type default) (color 0 0 0 0))
+  )
+  (wire (pts (xy 116.84 82.55) (xy 116.84 85.09))
+    (stroke (width 0) (type default) (color 0 0 0 0))
+  )
+  (global_label "3V3" (shape input) (at 53.34 77.47 180) (fields_autoplaced)
+    (effects (font (size 1.27 1.27)) (justify right))
+    (property "Intersheet References" "${INTERSHEET_REFS}" (id 0) (at 47.4193 77.3906 0)
+      (effects (font (size 1.27 1.27)) (justify right) hide)
+    )
+  )
+  (global_label "CURR-MONITOR" (shape input) (at 58.42 85.09 180) (fields_autoplaced)
+    (effects (font (size 1.27 1.27)) (justify right))
+    (property "Intersheet References" "${INTERSHEET_REFS}" (id 0) (at 41.0088 85.0106 0)
+      (effects (font (size 1.27 1.27)) (justify right) hide)
+    )
+  )
+  (global_label "3V3" (shape input) (at 119.38 87.63 180) (fields_autoplaced)
+    (effects (font (size 1.27 1.27)) (justify right))
+    (property "Intersheet References" "${INTERSHEET_REFS}" (id 0) (at 113.4593 87.5506 0)
+      (effects (font (size 1.27 1.27)) (justify right) hide)
+    )
+  )
+  (symbol (lib_id "Device:Ferrite_Bead_Small") (at 55.88 77.47 270) (unit 1)
+    (in_bom yes) (on_board yes)
+    (property "Reference" "FB?" (id 0) (at 55.88 71.4502 90))
+    (property "Value" "100R @ 100 MHz" (id 1) (at 53.34 73.66 90))
+    (property "Footprint" "STM32_Breakout:INDUC1607X60N" (id 2) (at 55.88 75.692 90)
+      (effects (font (size 1.27 1.27)) hide)
+    )
+    (property "Datasheet" "~" (id 3) (at 55.88 77.47 0)
+      (effects (font (size 1.27 1.27)) hide)
+    )
+    (pin "1")
+    (pin "2")
+  )
+  (symbol (lib_id "Connector:TestPoint") (at 119.38 85.09 270) (unit 1)
+    (in_bom yes) (on_board yes)
+    (property "Reference" "TP?" (id 0) (at 121.92 83.82 0)
+      (effects (font (size 1.27 1.27)) (justify right))
+    )
+    (property "Value" "TestPoint" (id 1) (at 124.46 88.9 0)
+      (effects (font (size 1.27 1.27)) (justify right))
+    )
+    (property "Footprint" "TestPoint:TestPoint_Pad_D2.0mm" (id 2) (at 119.38 90.17 0)
+      (effects (font (size 1.27 1.27)) hide)
+    )
+    (property "Datasheet" "~" (id 3) (at 119.38 90.17 0)
+      (effects (font (size 1.27 1.27)) hide)
+    )
+    (pin "1")
+  )
+  (symbol (lib_id "STM32_Breakout-rescue:MAX4372FESA+-MAX4372FESA+") (at 58.42 77.47 0) (unit 1)
+    (in_bom yes) (on_board yes)
+    (property "Reference" "MAX4372F?" (id 0) (at 86.36 67.6402 0)
+      (effects (font (size 1.524 1.524)))
+    )
+    (property "Value" "MAX4372FESA+" (id 1) (at 86.36 70.3326 0)
+      (effects (font (size 1.524 1.524)))
+    )
+    (property "Footprint" "STM32_Breakout:SOIC127P600X175-8N" (id 2) (at 69.85 63.5 0)
+      (effects (font (size 1.524 1.524)) hide)
+    )
+    (property "Datasheet" "" (id 3) (at 58.42 77.47 0)
+      (effects (font (size 1.524 1.524)))
+    )
+    (pin "1")
+    (pin "2")
+    (pin "3")
+    (pin "4")
+    (pin "5")
+    (pin "6")
+    (pin "7")
+    (pin "8")
+  )
+  (symbol (lib_id "power:GND") (at 58.42 82.55 270) (unit 1)
+    (in_bom yes) (on_board yes)
+    (property "Reference" "#PWR?" (id 0) (at 52.07 82.55 0)
+      (effects (font (size 1.27 1.27)) hide)
+    )
+    (property "Value" "GND" (id 1) (at 54.0258 82.677 0))
+    (property "Footprint" "" (id 2) (at 58.42 82.55 0)
+      (effects (font (size 1.27 1.27)) hide)
+    )
+    (property "Datasheet" "" (id 3) (at 58.42 82.55 0)
+      (effects (font (size 1.27 1.27)) hide)
+    )
+    (pin "1")
+  )
+  (symbol (lib_id "STM32_Breakout-rescue:R0603-OBC_Libary") (at 119.38 77.47 270) (unit 1)
+    (in_bom yes) (on_board yes)
+    (property "Reference" "R?" (id 0) (at 125.73 76.2 90)
+      (effects (font (size 1.27 1.27)) (justify left))
+    )
+    (property "Value" "20m" (id 1) (at 123.19 78.74 90)
+      (effects (font (size 1.27 1.27)) (justify left))
+    )
+    (property "Footprint" "RESC1607X60N" (id 2) (at 121.92 76.2 0)
+      (effects (font (size 1.27 1.27)) (justify left bottom) hide)
+    )
+    (property "Datasheet" "" (id 3) (at 119.38 77.47 0)
+      (effects (font (size 1.27 1.27)) (justify left bottom) hide)
+    )
+    (pin "1")
+    (pin "2")
+  )
 )

Commit message: comm-rfb: reformat main schematic page
Parts:
- gave numbers to parts that had none: 4
Changed lines of the file:
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@@
   (symbol (lib_id "Device:Ferrite_Bead_Small") (at 55.88 77.47 270) (unit 1)
     (in_bom yes) (on_board yes)
-    (property "Reference" "FB?" (id 0) (at 55.88 71.4502 90))
+    (property "Reference" "FB3" (id 0) (at 55.88 71.4502 90))
     (property "Value" "100R @ 100 MHz" (id 1) (at 53.34 73.66 90))
     (property "Footprint" "STM32_Breakout:INDUC1607X60N" (id 2) (at 55.88 75.692 90)
@@
   (symbol (lib_id "Connector:TestPoint") (at 119.38 85.09 270) (unit 1)
     (in_bom yes) (on_board yes)
-    (property "Reference" "TP?" (id 0) (at 121.92 83.82 0)
+    (property "Reference" "TP1" (id 0) (at 121.92 83.82 0)
       (effects (font (size 1.27 1.27)) (justify right))
     )
@@
   (symbol (lib_id "STM32_Breakout-rescue:MAX4372FESA+-MAX4372FESA+") (at 58.42 77.47 0) (unit 1)
     (in_bom yes) (on_board yes)
-    (property "Reference" "MAX4372F?" (id 0) (at 86.36 67.6402 0)
+    (property "Reference" "MAX4372F1" (id 0) (at 86.36 67.6402 0)
       (effects (font (size 1.524 1.524)))
     )
@@
   (symbol (lib_id "power:GND") (at 58.42 82.55 270) (unit 1)
     (in_bom yes) (on_board yes)
-    (property "Reference" "#PWR?" (id 0) (at 52.07 82.55 0)
+    (property "Reference" "#PWR019" (id 0) (at 52.07 82.55 0)
       (effects (font (size 1.27 1.27)) hide)
     )
@@
   (symbol (lib_id "STM32_Breakout-rescue:R0603-OBC_Libary") (at 119.38 77.47 270) (unit 1)
     (in_bom yes) (on_board yes)
-    (property "Reference" "R?" (id 0) (at 125.73 76.2 90)
+    (property "Reference" "R8" (id 0) (at 125.73 76.2 90)
       (effects (font (size 1.27 1.27)) (justify left))
     )
