File: ADCS_Boards/Controller_board/MC_SunSensorPCB.kicad_sch (KiCad schematic)
At the start: 106 parts, among them J1 PC104_Connector, J2 PPTC062LJBN-RC, J3 Conn_01x03_Female, Q12 20V/0.2A/8MHz/1.2Ω/1Vth, Q14 20V/0.2A/8MHz/1.2Ω/1Vth, Q3 20V/0.2A/8MHz/1.2Ω/1Vth, Q4 20V/0.2A/8MHz/1.2Ω/1Vth, Q6 20V/0.2A/8MHz/1.2Ω/1Vth, Q9 20V/0.2A/8MHz/1.2Ω/1Vth, U1 9DoF IMU, U10 Op-Amp, U11 Op-Amp, U12 Op-Amp, U13 Op-Amp, U14 1.8V/100mA, U15 STM32F103RET6, U16 MR25H10MDF, U2 1.8V/100mA, U3 9DoF IMU, U4 DF13-7P-1.25DS(20), U5 DF13-7P-1.25DS(20), U6 DF13-7P-1.25DS(20), U7 DF13-7P-1.25DS(20), U8 LM358, U9 CD74HC4067M96, Y1 Crystal_GND24

Commit message: adcs: Updated ADCS Controller board with latest status from Yasin
Parts:
- added C32, C34, C35, C36, C37, C38: 100n, Capacitor_SMD:C_0603_1608Metric, symbol Device:C
- added C33: 10u, Capacitor_SMD:C_0603_1608Metric, symbol Device:C
- added C39: 10n, Capacitor_SMD:C_0603_1608Metric, symbol Device:C
- added C40, C41: 1u, Capacitor_SMD:C_0603_1608Metric, symbol Device:C
- added FB2: FerriteBead, Inductor_SMD:L_0603_1608Metric, symbol Device:FerriteBead
- added R2: 10k, Resistor_SMD:R_0603_1608Metric, symbol Device:R
- added S1: TL3305CF260QG, Footprints_QSAT:SW_TL3305CF260QG, symbol ADCS_Symbols:TL3305CF260QG
- added U17: 1825232-1, Footprints_QSAT:1825232-1, symbol ADCS_Symbols:1825232-1
Connections:
- net +3V3: now also U15.1 (VBAT), U15.19 (VDD_4), U15.48 (VDD_2), U15.64 (VDD_3), C33.1, C34.1, C35.1, C36.1, C37.1, C38.1, C41.1, FB2.2, U17.3
- net GND: now also U15.12 (VSSA), U15.18 (VSS_4), U15.47 (VSS_2), U15.63 (VSS_3), C32.2, C33.2, C34.2, C35.2, C36.2, C37.2, C38.2, C39.2, C40.2, C41.2, S1.1, S1.2, U17.1
- net PD4_O3: no longer C17.1, R20.1, U11.9
- net PD4_O4: now also C17.1, R20.1, U11.9
- net +3.3VA: now reaches U15.13 (VDDA)
- net +3.3VA: now also C39.1, C40.1, FB2.1
- net BOOT0: now reaches U15.60 (BOOT0)
- net BOOT0: now also R2.2
- net NRST: now reaches U15.7 (NRST)
- net NRST: now also C32.1, S1.3, S1.4
- net Output_O1: no longer names the net of C4.1, R10.2, U10.7, U9.8 (I1)
- net Output_O2: no longer names the net of C15.1, R18.2, U13.7, U9.4 (I5)
- net Output_O3: no longer names the net of C13.1, R16.2, U12.7, U9.22 (I9)
- net Output_O4: no longer names the net of C11.1, R14.2, U11.7, U9.18 (I13)
- new net SW_BOOT0: R2.1, U17.2
Other:
- moved on the sheet: C31, D3, FB1, R53, R54, R55, U16
